File: BCInside/Strut.kicad_pcb (KiCad board)
At the start: 4 copper layers, 309.6 x 138.1 mm, 53 parts, among them J1 IN, J2 OUT

Commit message: First iteration of all struts
Parts:
- removed C16, C17: 100NF, Capacitor_SMD:C_0805_2012Metric
- removed D16, D17: WS2813, LED_SMD:LED_WS2812_PLCC6_5.0x5.0mm_P1.6mm
- removed R16, R17: 330, Resistor_SMD:R_0805_2012Metric
- moved C1 85.7 mm to (69.6, 67.3), turned to 180 degrees
- moved C9 82.0 mm to (200.7, 70.3), turned to 180 degrees
- moved J2 80.7 mm to (314.0, 72.4)
- moved C14 79.5 mm to (284.2, 69.8), turned to 180 degrees
- moved C15 79.2 mm to (301.2, 70.1), turned to 180 degrees
- moved R14 78.9 mm to (288.8, 69.8), turned to 180 degrees
- moved R15 78.7 mm to (305.1, 70.1), turned to 180 degrees
- moved J1 73.8 mm to (57.9, 72.6)
- moved R1 73.7 mm to (71.4, 70.1)
- moved C10 73.6 mm to (227.7, 75.0)
- moved C11 73.6 mm to (244.4, 75.0)
- moved C12 73.6 mm to (261.5, 75.0)
- moved C13 73.6 mm to (278.1, 75.0)
- moved C2 73.6 mm to (94.5, 75.0)
- moved C3 73.6 mm to (111.2, 75.0)
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Connections:
- J2 pad 2: Net-(D17-Pad3) -> Net-(D15-Pad3)
Routing:
- net Net-(D15-Pad3): track 36.1 -> 9.24 mm
- net Net-(D14-Pad3): track 31.6 -> 14.0 mm
- net Net-(D16-Pad3): track 13.5 -> 0.00 mm
- net Net-(C16-Pad1): track 12.3 -> 0.00 mm
- net Net-(C17-Pad1): track 11.8 -> 0.00 mm
- net Net-(D17-Pad3): track 9.86 -> 0.00 mm, vias 1 -> 0
- net +5V: track 89.0 -> 79.2 mm, vias 19 -> 20
- net Net-(C1-Pad1): track 15.6 -> 10.3 mm
- net Net-(C14-Pad1): track 6.15 -> 11.0 mm
- net Net-(C15-Pad1): track 6.15 -> 9.50 mm
- net GND: track 101.3 -> 98.2 mm, vias 20 -> 19
- net Net-(D10-Pad6): track 36.8 -> 33.9 mm
- net Net-(D13-Pad3): track 31.8 -> 34.5 mm
- net Net-(D1-Pad4): track 33.8 -> 31.3 mm
- net Net-(C9-Pad1): track 9.89 -> 9.22 mm, vias 2 -> 0
Other:
- outline, holes or cut-outs redrawn
