File: BCInside/BCInside.kicad_pcb (KiCad board)
At the start: 4 copper layers, 276.1 x 21.4 mm, 47 parts, among them J1 IN, J2 OUT

Commit message: Before changing Outside Struts to not have connectors
Parts:
- added J3: PWR_BRIDGE, YonaFootprints:TEDX_PWR_BRIDGE_TALL, B.Cu at (145.4, 145.3)
- added J3: PWR_BRIDGE, YonaFootprints:TEDX_PWR_BRIDGE_TALL, B.Cu at (112.1, 155.3)
- added J3: PWR_BRIDGE, YonaFootprints:TEDX_PWR_BRIDGE_TALL, B.Cu at (228.8, 155.3)
- added J3: PWR_BRIDGE, YonaFootprints:TEDX_PWR_BRIDGE_TALL, B.Cu at (262.1, 145.3)
- added J4: DAT_BRIDGE, YonaFootprints:TEDX_DAT_BRIDGE_TALL, B.Cu at (295.4, 145.3)
- added J5: OUT, YonaFootprints:TEDX_INNER_4, F.Cu at (310.0, 148.3)
- C1, C10, C11, C12, C13, C14, C15, C2, C3, C4, C5, C6, C7, C8, C9: value 100NF -> .1uF; footprint Capacitor_SMD:C_0805_2012Metric -> Capacitor_SMD:C_0603_1608Metric
- J1: footprint YonaFootprints:1x3_18awgWireSolderPad-InsideStrut -> YonaFootprints:TEDX_INNER_4
- J2: value OUT -> DAT_BRIDGE; footprint YonaFootprints:1x3_18awgWireSolderPad-InsideStrut-OUT -> YonaFootprints:TEDX_DAT_BRIDGE_TALL; moved to B.Cu
- R1, R10, R11, R12, R13, R14, R15, R2, R3, R4, R5, R6, R7, R8, R9: footprint Resistor_SMD:R_0805_2012Metric -> Resistor_SMD:R_0603_1608Metric
- moved J2 244.6 mm to (78.8, 155.3)
- moved C1 75.4 mm to (72.5, 143.3)
- moved J1 73.8 mm to (64.2, 148.3)
- moved D12 73.7 mm to (253.8, 148.3)
- moved D13 73.7 mm to (270.4, 148.3)
- moved D14 73.7 mm to (287.1, 148.3)
- moved D15 73.7 mm to (303.8, 148.3)
- moved D11 73.7 mm to (237.1, 148.3)
- moved D10 73.7 mm to (220.4, 148.3)
- moved D9 73.7 mm to (203.8, 148.3)
- moved D8 73.7 mm to (187.1, 148.3)
- moved D7 73.7 mm to (170.4, 148.3)
- moved D6 73.7 mm to (153.8, 148.3)
- moved D5 73.7 mm to (137.1, 148.3)
- moved D4 73.7 mm to (120.4, 148.3)
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Connections:
- net Net-(D1-Pad4) renamed /DIN
- net Net-(D14-Pad3) renamed /BOUT
- D1 pad 6: GND -> /BIN
- D15 pad 3: Net-(D15-Pad3) -> /DOUT
- J1 pad 3: GND -> /BIN
- J2 pad 1: +5V -> Net-(J2-Pad1)
- J2 pad 2: Net-(D15-Pad3) -> Net-(J2-Pad2)
Routing:
- net Net-(J2-Pad1): track 0.00 -> 258.2 mm, vias 0 -> 2
- net Net-(J2-Pad2): track 0.00 -> 248.4 mm
- net GND: track 89.0 -> 50.5 mm, vias 18 -> 30
- net +5V: track 77.8 -> 47.7 mm, vias 16 -> 27
- net /DOUT: track 0.00 -> 14.2 mm, vias 0 -> 3
- net /BOUT: track 14.0 -> 19.4 mm, vias 0 -> 2
- net Net-(D6-Pad3): track 32.1 -> 37.1 mm, vias 0 -> 4
- net Net-(D15-Pad3): track 4.83 -> 0.00 mm
- net Net-(D7-Pad3): track 31.9 -> 36.7 mm, vias 0 -> 4
- net Net-(C6-Pad1): track 5.93 -> 10.5 mm
- net Net-(C11-Pad1): track 5.93 -> 10.5 mm
- net Net-(C4-Pad1): track 5.93 -> 10.5 mm
- net Net-(C2-Pad1): track 5.93 -> 10.5 mm
- net Net-(C5-Pad1): track 5.93 -> 10.5 mm
- net Net-(D2-Pad3): track 32.1 -> 36.7 mm, vias 0 -> 4
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- removed copper zone on In2.Cu, net +5V
- removed copper zone on In1.Cu, net GND
Other:
- board size 276.1 x 21.4 mm -> 276.2 x 21.6 mm
- copper layers 4 -> 2
- board text added: "5v"
- board text added: "BIN"
- board text added: "BOUT"
- board text added: "C/O BO"
- board text added: "C/O DO"
- board text added: "C/O IN"
- board text added: "DIN"
- board text added: "DOUT"
- board text added: "G"
- board text added: "GND"

Commit message: Prototype v4
Routing:
- net Net-(J2-Pad1): track 258.2 -> 247.5 mm, vias 2 -> 0
- net Net-(J2-Pad2): track 248.4 -> 250.8 mm
Changed lines of the file:
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@@
     (thickness 1.6)
     (drawings 218)
-    (tracks 564)
+    (tracks 558)
     (zones 0)
     (modules 53)
@@
     (last_trace_width 0.3)
     (trace_clearance 0.25)
-    (zone_clearance 0.508)
+    (zone_clearance 0.381)
     (zone_45_only no)
     (trace_min 0.2)
@@
   (segment (start 81.145 146.696) (end 80.444999 145.995999) (width 0.3) (layer F.Cu) (net 18))
   (segment (start 80.444999 145.995999) (end 79.945 145.496) (width 0.3) (layer F.Cu) (net 18))
-  (segment (start 74.545 146.696) (end 74.745005 146.495995) (width 0.3) (layer F.Cu) (net 18))
-  (via (at 74.745005 146.495995) (size 1) (drill 0.6) (layers F.Cu B.Cu) (net 18))
-  (segment (start 75.745 145.496) (end 75.245004 145.995996) (width 0.3) (layer B.Cu) (net 18))
-  (segment (start 72.895 146.696) (end 74.545 146.696) (width 0.3) (layer F.Cu) (net 18))
-  (segment (start 79.945 145.496) (end 75.745 145.496) (width 0.3) (layer B.Cu) (net 18))
-  (segment (start 75.245004 145.995996) (end 74.745005 146.495995) (width 0.3) (layer B.Cu) (net 18))
+  (via (at 74.745 145.496001) (size 1) (drill 0.6) (layers F.Cu B.Cu) (net 18))
+  (segment (start 75.452106 145.496001) (end 74.745 145.496001) (width 0.3) (layer B.Cu) (net 18))
+  (segment (start 79.945 145.496) (end 79.237893 145.496001) (width 0.3) (layer B.Cu) (net 18))
+  (segment (start 73.145 146.696) (end 74.344999 145.496001) (width 0.3) (layer F.Cu) (net 18))
+  (segment (start 72.895 146.696) (end 73.145 146.696) (width 0.3) (layer F.Cu) (net 18))
+  (segment (start 79.237893 145.496001) (end 75.452106 145.496001) (width 0.3) (layer B.Cu) (net 18))
+  (segment (start 74.344999 145.496001) (end 74.745 145.496001) (width 0.3) (layer F.Cu) (net 18))
   (via (at 130.94406 152.496) (size 1) (drill 0.6) (layers F.Cu B.Cu) (net 19))
   (via (at 122.3774 152.496) (size 1) (drill 0.6) (layers F.Cu B.Cu) (net 19))
@@
   (segment (start 70.227 146.696) (end 70.944997 147.413997) (width 0.3) (layer F.Cu) (net 32))
   (segment (start 70.944997 147.413997) (end 70.944997 149.096001) (width 0.3) (layer F.Cu) (net 32))
+  (segment (start 78.945 149.096) (end 74.394999 153.646001) (width 0.3) (layer F.Cu) (net 32))
   (segment (start 70.444998 154.095998) (end 70.495 154.146) (width 0.3) (layer B.Cu) (net 32))
+  (via (at 70.495 154.146) (size 1) (drill 0.6) (layers F.Cu B.Cu) (net 32))
   (segment (start 70.444998 149.596) (end 70.444998 154.095998) (width 0.3) (layer B.Cu) (net 32))
-  (via (at 70.495 154.146) (size 1) (drill 0.6) (layers F.Cu B.Cu) (net 32))
-  (segment (start 70.994999 153.646001) (end 70.495 154.146) (width 0.3) (layer F.Cu) (net 32))
-  (segment (start 74.394999 153.646001) (end 70.994999 153.646001) (width 0.3) (layer F.Cu) (net 32))
-  (segment (start 82.545 149.096) (end 78.945 149.096) (width 0.3) (layer F.Cu) (net 32))
-  (segment (start 78.945 149.096) (end 74.394999 153.646001) (width 0.3) (layer F.Cu) (net 32))
   (segment (start 83.345 149.896) (end 82.545 149.096) (width 0.3) (layer F.Cu) (net 32))
   (segment (start 84.66166 149.896) (end 83.345 149.896) (width 0.3) (layer F.Cu) (net 32))
+  (segment (start 82.545 149.096) (end 78.945 149.096) (width 0.3) (layer F.Cu) (net 32))
+  (segment (start 74.394999 153.646001) (end 70.994999 153.646001) (width 0.3) (layer F.Cu) (net 32))
+  (segment (start 70.994999 153.646001) (end 70.495 154.146) (width 0.3) (layer F.Cu) (net 32))
   (segment (start 298.2118 146.696) (end 297.7118 146.196) (width 0.3) (layer F.Cu) (net 33))
   (via (at 297.7118 146.196) (size 1) (drill 0.6) (layers F.Cu B.Cu) (net 33))
@@
   (segment (start 304.852106 146.696) (end 304.145 146.696) (width 0.3) (layer F.Cu) (net 34))
   (segment (start 309.152375 149.296) (end 310.027375 149.296) (width 0.3) (layer B.Cu) (net 35))
+  (segment (start 81.027549 155.778549) (end 81.027549 153.296) (width 0.3) (layer B.Cu) (net 35))
+  (segment (start 310.367168 155.896) (end 81.145 155.896) (width 0.3) (layer B.Cu) (net 35))
+  (segment (start 312.052364 154.210804) (end 310.367168 155.896) (width 0.3) (layer B.Cu) (net 35))
+  (segment (start 81.145 155.896) (end 81.027549 155.778549) (width 0.3) (layer B.Cu) (net 35))
+  (segment (start 312.052364 150.445989) (end 312.052364 154.210804) (width 0.3) (layer B.Cu) (net 35))
+  (segment (start 310.902375 149.296) (end 312.052364 150.445989) (width 0.3) (layer B.Cu) (net 35))
   (segment (start 310.027375 149.296) (end 310.902375 149.296) (width 0.3) (layer B.Cu) (net 35))
-  (segment (start 310.902375 149.296) (end 312.052364 150.445989) (width 0.3) (layer B.Cu) (net 35))
-  (segment (start 312.052364 150.445989) (end 312.052364 154.210804) (width 0.3) (layer B.Cu) (net 35))
-  (segment (start 312.052364 154.210804) (end 310.367168 155.896) (width 0.3) (layer B.Cu) (net 35))
-  (segment (start 81.027549 155.813451) (end 81.027549 153.296) (width 0.3) (layer B.Cu) (net 35))
-  (segment (start 310.367168 155.896) (end 80.945 155.896) (width 0.3) (layer B.Cu) (net 35))
-  (segment (start 80.945 155.896) (end 81.027549 155.813451) (width 0.3) (layer B.Cu) (net 35))
-  (segment (start 76.527549 155.478549) (end 76.527549 153.296) (width 0.3) (layer B.Cu) (net 35))
-  (segment (start 76.945 155.896) (end 76.527549 155.478549) (width 0.3) (layer B.Cu) (net 35))
-  (segment (start 80.945 155.896) (end 76.945 155.896) (width 0.3) (layer B.Cu) (net 35))
+  (segment (start 80.945 150.796) (end 76.645 150.796) (width 0.3) (layer B.Cu) (net 35))
+  (segment (start 76.645 150.796) (end 76.527549 150.913451) (width 0.3) (layer B.Cu) (net 35))
+  (segment (start 81.027549 150.878549) (end 80.945 150.796) (width 0.3) (layer B.Cu) (net 35))
+  (segment (start 76.527549 150.913451) (end 76.527549 153.296) (width 0.3) (layer B.Cu) (net 35))
+  (segment (start 81.027549 153.296) (end 81.027549 150.878549) (width 0.3) (layer B.Cu) (net 35))
   (segment (start 311.1118 147.296) (end 310.027375 147.296) (width 0.3) (layer B.Cu) (net 36))
-  (via (at 79.035913 150.677895) (size 1) (drill 0.6) (layers F.Cu B.Cu) (net 36))
-  (segment (start 78.777549 150.936259) (end 79.035913 150.677895) (width 0.3) (layer B.Cu) (net 36))
-  (segment (start 78.777549 153.296) (end 78.777549 150.936259) (width 0.3) (layer B.Cu) (net 36))
-  (via (at 75.045 155.396) (size 1) (drill 0.6) (layers F.Cu B.Cu) (net 36))
+  (segment (start 78.777549 156.128549) (end 78.777549 153.296) (width 0.3) (layer B.Cu) (net 36))
+  (segment (start 79.144999 156.495999) (end 78.777549 156.128549) (width 0.3) (layer B.Cu) (net 36))
+  (segment (start 310.545001 156.495999) (end 79.144999 156.495999) (width 0.3) (layer B.Cu) (net 36))
+  (segment (start 312.602375 154.438625) (end 310.545001 156.495999) (width 0.3) (layer B.Cu) (net 36))
+  (segment (start 310.027375 147.296) (end 310.902375 147.296) (width 0.3) (layer B.Cu) (net 36))
   (segment (start 312.602375 148.996) (end 312.602375 154.438625) (width 0.3) (layer B.Cu) (net 36))
-  (segment (start 310.545001 156.495999) (end 76.144999 156.495999) (width 0.3) (layer B.Cu) (net 36))
-  (segment (start 310.027375 147.296) (end 310.902375 147.296) (width 0.3) (layer B.Cu) (net 36))
   (segment (start 310.902375 147.296) (end 312.602375 148.996) (width 0.3) (layer B.Cu) (net 36))
-  (segment (start 312.602375 154.438625) (end 310.545001 156.495999) (width 0.3) (layer B.Cu) (net 36))
-  (segment (start 76.144999 156.495999) (end 75.544999 155.895999) (width 0.3) (layer B.Cu) (net 36))
-  (segment (start 75.544999 155.895999) (end 75.045 155.396) (width 0.3) (layer B.Cu) (net 36))
-  (segment (start 75.845 155.396) (end 75.045 155.396) (width 0.3) (layer F.Cu) (net 36))
-  (segment (start 76.345 154.896) (end 75.845 155.396) (width 0.3) (layer F.Cu) (net 36))
-  (segment (start 76.345 154.796) (end 76.345 154.896) (width 0.3) (layer F.Cu) (net 36))
-  (segment (start 79.035913 152.105087) (end 76.345 154.796) (width 0.3) (layer F.Cu) (net 36))
-  (segment (start 79.035913 150.677895) (end 79.035913 152.105087) (width 0.3) (layer F.Cu) (net 36))
   (zone (net 2) (net_name GND) (layer B.Cu) (hatch edge 0.508)
-    (connect_pads (clearance 0.508))
+    (connect_pads (clearance 0.381))
     (min_thickness 0.254)
     (fill yes (arc_segments 16) (thermal_gap 0.508) (thermal_bridge_width 0.508))
@@
   )
   (zone (net 1) (net_name +5V) (layer F.Cu) (hatch edge 0.508)
-    (connect_pads (clearance 0.508))
+    (connect_pads (clearance 0.381))
     (min_thickness 0.254)
     (fill yes (arc_segments 16) (thermal_gap 0.508) (thermal_bridge_width 0.508))
