File: BCOutside/Strut.kicad_pcb (KiCad board)
At the start: 4 copper layers, 309.6 x 138.1 mm, 53 parts, among them J1 IN, J2 OUT

Commit message: First iteration of all struts
Parts:
- removed C16, C17: 100NF, Capacitor_SMD:C_0805_2012Metric
- removed D16, D17: WS2813, LED_SMD:LED_WS2812_PLCC6_5.0x5.0mm_P1.6mm
- removed R16, R17: 330, Resistor_SMD:R_0805_2012Metric
- moved J2 64.9 mm to (314.8, 89.7)
- moved C1 61.1 mm to (78.5, 92.1), turned to 90 degrees
- moved C9 60.4 mm to (212.3, 92.1), turned to 90 degrees
- moved C15 58.2 mm to (297.7, 92.1)
- moved J1 56.7 mm to (57.7, 89.7)
- moved R15 56.6 mm to (307.9, 92.1)
- moved C10 56.5 mm to (227.7, 92.1)
- moved C11 56.5 mm to (244.4, 92.1)
- moved C12 56.5 mm to (261.5, 92.1)
- moved C13 56.5 mm to (278.1, 92.1)
- moved C14 56.5 mm to (294.8, 92.1)
- moved C2 56.5 mm to (94.5, 92.1)
- moved C3 56.5 mm to (111.2, 92.1)
- moved C4 56.5 mm to (127.8, 92.1)
- moved C5 56.5 mm to (144.5, 92.1)
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Connections:
- J2 pad 2: Net-(D17-Pad3) -> Net-(D15-Pad3)
Routing:
- net Net-(D15-Pad3): track 36.1 -> 10.1 mm
- net Net-(D14-Pad3): track 31.6 -> 12.6 mm
- net GND: track 101.3 -> 117.2 mm, vias 20 -> 16
- net Net-(D16-Pad3): track 13.5 -> 0.00 mm
- net Net-(C16-Pad1): track 12.3 -> 0.00 mm
- net Net-(C17-Pad1): track 11.8 -> 0.00 mm
- net Net-(D17-Pad3): track 9.86 -> 0.00 mm, vias 1 -> 0
- net Net-(C1-Pad1): track 15.6 -> 6.56 mm
- net Net-(C15-Pad1): track 6.15 -> 11.2 mm, vias 0 -> 2
- net Net-(D10-Pad6): track 36.8 -> 32.6 mm
- net +5V: track 89.0 -> 92.4 mm, vias 19 -> 17
- net Net-(D1-Pad4): track 33.8 -> 30.4 mm
- net Net-(C9-Pad1): track 9.89 -> 7.09 mm, vias 2 -> 0
- net Net-(D1-Pad3): track 34.0 -> 31.9 mm
- net Net-(D10-Pad4): track 33.7 -> 32.6 mm
Other:
- outline, holes or cut-outs redrawn
