File: DInside/Strut.kicad_pcb (KiCad board)
At the start: 4 copper layers, 309.6 x 138.1 mm, 53 parts, among them J1 IN, J2 OUT

Commit message: First iteration of all struts
Parts:
- removed C17: 100NF, Capacitor_SMD:C_0805_2012Metric
- removed D17: WS2813, LED_SMD:LED_WS2812_PLCC6_5.0x5.0mm_P1.6mm
- removed R17: 330, Resistor_SMD:R_0805_2012Metric
- moved C1 50.0 mm to (69.6, 103.0), turned to 180 degrees
- moved C16 47.3 mm to (315.9, 105.9), turned to 180 degrees
- moved C9 46.4 mm to (200.7, 106.1), turned to 180 degrees
- moved C15 44.0 mm to (301.2, 105.8), turned to 180 degrees
- moved R15 43.0 mm to (305.1, 105.8), turned to 180 degrees
- moved J2 41.3 mm to (331.4, 107.9)
- moved J1 38.1 mm to (57.9, 108.3)
- moved R1 38.0 mm to (71.4, 105.8)
- moved C10 37.9 mm to (227.7, 110.8)
- moved C11 37.9 mm to (244.4, 110.8)
- moved C12 37.9 mm to (261.5, 110.8)
- moved C13 37.9 mm to (278.1, 110.8)
- moved C14 37.9 mm to (294.8, 110.8)
- moved C2 37.9 mm to (94.5, 110.8)
- moved C3 37.9 mm to (111.2, 110.8)
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Connections:
- J2 pad 2: Net-(D17-Pad3) -> Net-(D16-Pad3)
Routing:
- net Net-(D15-Pad3): track 36.1 -> 13.0 mm
- net Net-(C17-Pad1): track 11.8 -> 0.00 mm
- net Net-(D17-Pad3): track 9.86 -> 0.00 mm, vias 1 -> 0
- net Net-(C1-Pad1): track 15.6 -> 10.3 mm
- net Net-(D10-Pad6): track 36.8 -> 33.0 mm
- net Net-(D16-Pad3): track 13.5 -> 9.85 mm
- net Net-(C15-Pad1): track 6.15 -> 9.50 mm
- net Net-(D1-Pad4): track 33.8 -> 30.4 mm
- net Net-(C16-Pad1): track 12.3 -> 10.4 mm
- net GND: track 101.3 -> 103.1 mm
- net Net-(C9-Pad1): track 9.89 -> 9.22 mm, vias 2 -> 0
- net +5V: track 89.0 -> 88.7 mm, vias 19 -> 20
Other:
- outline, holes or cut-outs redrawn
