File: DInside/DInside.sch (KiCad schematic (older format))
At the start: 50 parts, among them J1 IN, J2 OUT

Commit message: Before changing Outside Struts to not have connectors
Parts:
- removed J1: IN, YonaFootprints:1x3_18awgWireSolderPad-InsideStrut, symbol Connector:Conn_01x03_Male
- removed J2: OUT, YonaFootprints:1x3_18awgWireSolderPad-InsideStrut-OUT, symbol Connector:Conn_01x03_Female
- added J1: IN, YonaFootprints:TEDX_INNER_4, symbol Connector:Conn_01x04_Male
- added J2: CO_BRIDGE, YonaFootprints:TEDX_DAT_BRIDGE_TALL, symbol Connector:Conn_01x02_Female
- added J3: PWR_BRIDGE, YonaFootprints:TEDX_PWR_BRIDGE_TALL, symbol Connector:Conn_01x02_Male
- added J4: DAT_BRIDGE, YonaFootprints:TEDX_DAT_BRIDGE_TALL, symbol Connector:Conn_01x02_Female
- added J5: OUT, YonaFootprints:TEDX_INNER_4, symbol Connector:Conn_01x04_Female
- C1, C10, C11, C12, C13, C14, C15, C16, C2, C3, C4, C5, C6, C7, C8, C9: value 100NF -> .1uF; footprint Capacitor_SMD:C_0805_2012Metric -> Capacitor_SMD:C_0603_1608Metric
- R1, R10, R11, R12, R13, R14, R15, R16, R2, R3, R4, R5, R6, R7, R8, R9: footprint Resistor_SMD:R_0805_2012Metric -> Resistor_SMD:R_0603_1608Metric
Connections:
- net labels added: BIN, BOUT, DIN, DOUT
- wire segments 275 -> 279
Other:
- note added: "D Strut\n15 LEDs"
- note removed: "E Strut\n17 LEDs\nx3"
- moved on the sheet: C1, D1, R1
