File: DInside/DInside.kicad_pcb (KiCad board)
At the start: 4 copper layers, 294.9 x 21.4 mm, 50 parts, among them J1 IN, J2 OUT

Commit message: Before changing Outside Struts to not have connectors
Parts:
- added J3: PWR_BRIDGE, YonaFootprints:TEDX_PWR_BRIDGE_TALL, B.Cu at (161.3, 145.2)
- added J3: PWR_BRIDGE, YonaFootprints:TEDX_PWR_BRIDGE_TALL, B.Cu at (111.3, 155.2)
- added J3: PWR_BRIDGE, YonaFootprints:TEDX_PWR_BRIDGE_TALL, B.Cu at (227.9, 155.2)
- added J3: PWR_BRIDGE, YonaFootprints:TEDX_PWR_BRIDGE_TALL, B.Cu at (277.9, 145.2)
- added J4: DAT_BRIDGE, YonaFootprints:TEDX_DAT_BRIDGE_TALL, B.Cu at (311.3, 145.2)
- added J5: OUT, YonaFootprints:TEDX_INNER_4, F.Cu at (325.9, 148.2)
- C1, C10, C11, C12, C13, C14, C15, C16, C2, C3, C4, C5, C6, C7, C8, C9: value 100NF -> .1uF; footprint Capacitor_SMD:C_0805_2012Metric -> Capacitor_SMD:C_0603_1608Metric
- J1: footprint YonaFootprints:1x3_18awgWireSolderPad-InsideStrut -> YonaFootprints:TEDX_INNER_4
- J2: value OUT -> CO_BRIDGE; footprint YonaFootprints:1x3_18awgWireSolderPad-InsideStrut-OUT -> YonaFootprints:TEDX_DAT_BRIDGE_TALL; moved to B.Cu
- R1, R10, R11, R12, R13, R14, R15, R16, R2, R3, R4, R5, R6, R7, R8, R9: footprint Resistor_SMD:R_0805_2012Metric -> Resistor_SMD:R_0603_1608Metric
- moved J2 252.7 mm to (77.9, 155.2)
- moved J1 38.2 mm to (63.4, 148.3)
- moved D12 37.9 mm to (252.9, 148.2)
- moved D13 37.9 mm to (269.6, 148.2)
- moved D14 37.9 mm to (286.3, 148.2)
- moved D15 37.9 mm to (302.9, 148.2)
- moved D16 37.9 mm to (319.6, 148.2)
- moved D11 37.9 mm to (236.3, 148.2)
- moved D10 37.9 mm to (219.6, 148.2)
- moved D9 37.9 mm to (202.9, 148.2)
- moved D8 37.9 mm to (186.3, 148.2)
- moved D7 37.9 mm to (169.6, 148.2)
- moved D6 37.9 mm to (152.9, 148.2)
- moved D5 37.9 mm to (136.3, 148.2)
- moved D4 37.9 mm to (119.6, 148.2)
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Connections:
- net Net-(D1-Pad4) renamed /DIN
- net Net-(D15-Pad3) renamed /BOUT
- D1 pad 6: GND -> /BIN
- D16 pad 3: Net-(D16-Pad3) -> /DOUT
- J1 pad 3: GND -> /BIN
- J2 pad 1: +5V -> Net-(J2-Pad1)
- J2 pad 2: Net-(D16-Pad3) -> Net-(J2-Pad2)
Routing:
- net Net-(J2-Pad2): track 0.00 -> 266.5 mm
- net Net-(J2-Pad1): track 0.00 -> 262.3 mm
- net GND: track 93.0 -> 49.1 mm, vias 19 -> 32
- net +5V: track 80.3 -> 52.1 mm, vias 19 -> 31
- net /DOUT: track 0.00 -> 14.2 mm, vias 0 -> 3
- net /BOUT: track 13.2 -> 19.6 mm, vias 0 -> 2
- net Net-(D16-Pad3): track 5.21 -> 0.00 mm
- net Net-(C6-Pad1): track 5.93 -> 10.5 mm
- net Net-(C11-Pad1): track 5.93 -> 10.5 mm
- net Net-(C4-Pad1): track 5.93 -> 10.5 mm
- net Net-(C2-Pad1): track 5.93 -> 10.5 mm
- net Net-(C5-Pad1): track 5.93 -> 10.5 mm
- net Net-(C14-Pad1): track 6.15 -> 10.5 mm
- net Net-(C8-Pad1): track 5.93 -> 10.3 mm
- net Net-(C13-Pad1): track 6.15 -> 10.5 mm
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- removed copper zone on In2.Cu, net +5V
- removed copper zone on In1.Cu, net GND
Other:
- board size 294.9 x 21.4 mm -> 295 x 21.5 mm
- copper layers 4 -> 2
- board text added: "5v"
- board text added: "B"
- board text added: "BIN"
- board text added: "BOUT"
- board text added: "C/O BO"
- board text added: "C/O DO"
- board text added: "C/O IN"
- board text added: "DIN"
- board text added: "DO"
- board text added: "DOUT"
- board text added: "G"
- board text added: "GND"

Commit message: Prototype v4
Routing:
- net +5V: track 52.1 -> 52.7 mm
Changed lines of the file:
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@@
   (segment (start 166.733767 143.237) (end 166.7 143.270767) (width 0.3) (layer F.Cu) (net 1))
   (segment (start 166.7 143.892894) (end 166.7 144.6) (width 0.3) (layer F.Cu) (net 1))
-  (segment (start 161.308691 144.531436) (end 161.308691 145.238542) (width 0.5) (layer B.Cu) (net 1))
-  (segment (start 161.271345 144.237) (end 161.308691 144.274346) (width 0.5) (layer B.Cu) (net 1))
-  (via (at 161.308691 145.238542) (size 1) (drill 0.6) (layers F.Cu B.Cu) (net 1))
-  (segment (start 161.308691 144.274346) (end 161.308691 144.531436) (width 0.5) (layer B.Cu) (net 1))
   (via (at 278.153134 145.680326) (size 1) (drill 0.6) (layers F.Cu B.Cu) (net 1))
   (via (at 283.299998 144.699998) (size 1) (drill 0.6) (layers F.Cu B.Cu) (net 1))
@@
   (segment (start 200.067447 143.237) (end 198.663 143.237) (width 0.3) (layer F.Cu) (net 1))
   (via (at 198.6 143.3) (size 1) (drill 0.6) (layers F.Cu B.Cu) (net 1))
+  (via (at 161.4 145.8) (size 1) (drill 0.6) (layers F.Cu B.Cu) (net 1))
+  (segment (start 161.271345 144.237) (end 161.4 144.365655) (width 0.5) (layer B.Cu) (net 1))
+  (segment (start 161.4 144.365655) (end 161.4 145.092894) (width 0.5) (layer B.Cu) (net 1))
+  (segment (start 161.4 145.092894) (end 161.4 145.8) (width 0.5) (layer B.Cu) (net 1))
   (via (at 307.104064 143.237) (size 1) (drill 0.6) (layers F.Cu B.Cu) (net 2))
   (segment (start 255.808433 143.237) (end 257.104264 143.237) (width 0.3) (layer F.Cu) (net 2))
