File: EOutside/Strut.kicad_pcb (KiCad board)
At the start: 4 copper layers, 309.6 x 138.1 mm, 53 parts, among them J1 IN, J2 OUT

Commit message: First iteration of all struts
Parts:
- moved R17 25.2 mm to (342.4, 169.2)
- moved J1 19.5 mm to (58.2, 165.6)
- moved C1 19.4 mm to (77.4, 167.7)
- moved C10 19.4 mm to (227.7, 168.1)
- moved C11 19.4 mm to (244.4, 168.1)
- moved C12 19.4 mm to (261.5, 168.1)
- moved C13 19.4 mm to (278.1, 168.1)
- moved C14 19.4 mm to (294.8, 168.1)
- moved C15 19.4 mm to (311.4, 168.1)
- moved C16 19.4 mm to (328.1, 168.1)
- moved C2 19.4 mm to (94.5, 168.1)
- moved C3 19.4 mm to (111.2, 168.1)
- moved C4 19.4 mm to (127.8, 168.1)
- moved C5 19.4 mm to (144.5, 168.1)
- moved C6 19.4 mm to (161.1, 168.1)
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Routing:
- net Net-(C17-Pad1): track 11.8 -> 5.06 mm
- net +5V: track 87.9 -> 82.1 mm, vias 16 -> 18
- net Net-(D1-Pad4): track 26.9 -> 29.8 mm
- net Net-(C16-Pad1): track 3.41 -> 6.15 mm
- net Net-(D17-Pad3): track 9.86 -> 10.7 mm
- net GND: vias 17 -> 18
Other:
- board size 309.6 x 138.1 mm -> 306.4 x 6 mm
