File: EOutside/EOutside.kicad_pcb (KiCad board)
At the start: 4 copper layers, 250 x 6.5 mm, 74 parts, among them J1 IN, J2 MID, J3 MID, J4 MID, J5 OUT, J6 PWR_BRIDGE

Commit message: Second Prototype Run
Parts:
- removed the J6 at (258.3, 104.8)
- removed the J6 at (75.0, 104.5)
- removed the J6 at (75.0, 98.2)
- removed the J6 at (91.7, 98.2)
- removed the J6 at (91.7, 104.8)
- removed the J6 at (108.3, 104.8)
- removed the J6 at (108.3, 98.2)
- removed the J6 at (125.0, 104.5)
- removed the J6 at (125.0, 98.2)
- removed the J6 at (141.7, 104.8)
- removed the J6 at (258.3, 98.2)
- removed the J6 at (141.7, 98.2)
- added J10: DAT_BRIDGE, YonaFootprints:TEDX_DAT_BRIDGE, B.Cu at (291.7, 104.8)
- added J10: DAT_BRIDGE, YonaFootprints:TEDX_DAT_BRIDGE, B.Cu at (291.7, 100.8)
- added J11: DAT_BRIDGE, YonaFootprints:TEDX_DAT_BRIDGE, B.Cu at (308.3, 104.8)
- added J11: DAT_BRIDGE, YonaFootprints:TEDX_DAT_BRIDGE, B.Cu at (308.3, 100.8)
- added J6: PWR_BRIDGE, YonaFootprints:TEDX_PWR_BRIDGE, F.Cu at (233.3, 98.2)
- added J6: PWR_BRIDGE, YonaFootprints:TEDX_PWR_BRIDGE, F.Cu at (116.7, 98.2)
- added J7: DAT_BRIDGE, YonaFootprints:TEDX_DAT_BRIDGE, F.Cu at (83.3, 98.2)
- added J7: DAT_BRIDGE, YonaFootprints:TEDX_DAT_BRIDGE, B.Cu at (75.0, 104.8)
- added J7: DAT_BRIDGE, YonaFootprints:TEDX_DAT_BRIDGE, B.Cu at (75.0, 98.2)
- added J8: DAT_BRIDGE, YonaFootprints:TEDX_DAT_BRIDGE, B.Cu at (258.3, 104.8)
- added J8: DAT_BRIDGE, YonaFootprints:TEDX_DAT_BRIDGE, B.Cu at (258.3, 100.7)
- added J9: DAT_BRIDGE, YonaFootprints:TEDX_DAT_BRIDGE, B.Cu at (275.0, 104.8)
- added J9: DAT_BRIDGE, YonaFootprints:TEDX_DAT_BRIDGE, B.Cu at (275.0, 100.8)
- moved R1 6.03 mm to (85.7, 103.1), turned to 180 degrees
- moved C3 4.58 mm to (119.3, 103.0), turned to 0 degrees
- moved C10 4.01 mm to (235.2, 103.2), turned to 0 degrees
- moved R3 3.19 mm to (116.0, 103.0), turned to 0 degrees
- moved R10 2.63 mm to (231.7, 103.2), turned to 0 degrees
- moved C1 1.78 mm to (81.8, 103.1), turned to 180 degrees
- moved C12 1.04 mm to (253.0, 103.2), turned to 180 degrees
- moved C13 0.30 mm to (270.5, 102.8)
- moved C14 0.30 mm to (287.2, 102.8)
- moved R13 0.30 mm to (279.6, 102.8)
- moved R14 0.30 mm to (296.2, 102.8)
- moved R15 0.30 mm to (312.9, 102.8)
- moved C15 0.29 mm to (303.8, 102.8)
- moved J1 0.26 mm to (67.9, 101.5)
- moved J5 0.25 mm to (315.4, 101.5)
Routing:
- net +5V: track 229.7 -> 153.2 mm
- net Net-(D1-Pad6): track 4.74 -> 43.6 mm, vias 0 -> 3
- net Net-(D11-Pad3): track 34.8 -> 52.9 mm, vias 2 -> 3
- net Net-(D12-Pad3): track 38.0 -> 55.2 mm, vias 2 -> 4
- net Net-(D14-Pad3): track 26.5 -> 41.7 mm, vias 2 -> 4
- net Net-(D13-Pad3): track 37.7 -> 51.5 mm, vias 3 -> 4
- net Net-(D1-Pad4): track 22.7 -> 35.8 mm, vias 2 -> 4
- net GND: track 144.2 -> 153.6 mm, vias 26 -> 24
- net Net-(D1-Pad3): track 29.9 -> 36.8 mm
- net Net-(D10-Pad3): track 31.8 -> 37.6 mm, vias 2 -> 4
- net Net-(D2-Pad3): track 29.9 -> 35.2 mm
- net Net-(D3-Pad3): track 29.9 -> 35.0 mm, vias 2 -> 3
- net Net-(D15-Pad3): track 8.11 -> 12.4 mm, vias 1 -> 2
- net Net-(C1-Pad1): track 4.63 -> 8.54 mm
- net Net-(C3-Pad1): track 4.63 -> 8.36 mm
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Other:
- board text added: "BI"
- board text added: "BIN"
- board text added: "BO"
- board text added: "DI"
- board text added: "DIN"
- board text added: "DO"
- board text added: "G"

Commit message: Before changing Outside Struts to not have connectors
Parts:
- added C16: .1uF, Capacitor_SMD:C_0603_1608Metric, F.Cu at (320.5, 102.8)
- added C17: .1uF, Capacitor_SMD:C_0603_1608Metric, F.Cu at (337.1, 102.8)
- added D16: WS2813, LED_SMD:LED_WS2812_PLCC6_5.0x5.0mm_P1.6mm, F.Cu at (325.0, 101.5)
- added D17: WS2813, LED_SMD:LED_WS2812_PLCC6_5.0x5.0mm_P1.6mm, F.Cu at (341.7, 101.5)
- added J12: MID, YonaFootprints:6mmStripMid, F.Cu at (333.3, 101.5)
- added J13: OUT, YonaFootprints:6mmStripEnd, F.Cu at (348.7, 101.5)
- added J14: DAT_BRIDGE, YonaFootprints:TEDX_DAT_BRIDGE, B.Cu at (325.0, 100.8)
- added J14: DAT_BRIDGE, YonaFootprints:TEDX_DAT_BRIDGE, B.Cu at (325.0, 104.8)
- added J15: DAT_BRIDGE, YonaFootprints:TEDX_DAT_BRIDGE, B.Cu at (341.7, 100.8)
- added J15: DAT_BRIDGE, YonaFootprints:TEDX_DAT_BRIDGE, B.Cu at (341.7, 104.8)
- added R16: 330, Resistor_SMD:R_0603_1608Metric, F.Cu at (329.6, 102.8)
- added R17: 330, Resistor_SMD:R_0603_1608Metric, F.Cu at (346.2, 102.8)
- J5: value OUT -> MID; footprint YonaFootprints:6mmStripEnd -> YonaFootprints:6mmStripMid
- moved J5 1.25 mm to (316.7, 101.5)
Routing:
- net Net-(D16-Pad3): track 0.00 -> 41.6 mm, vias 0 -> 4
- net Net-(D15-Pad3): track 12.4 -> 50.8 mm, vias 2 -> 4
- net GND: track 153.6 -> 167.4 mm, vias 24 -> 26
- net +5V: track 153.2 -> 167.1 mm
- net Net-(D17-Pad3): track 0.00 -> 12.5 mm, vias 0 -> 2
- net Net-(C17-Pad1): track 0.00 -> 10.5 mm
- net Net-(C16-Pad1): track 0.00 -> 10.5 mm
- net Net-(D14-Pad3): track 41.7 -> 52.0 mm
Other:
- board size 250 x 6.5 mm -> 283.3 x 6.5 mm

Commit message: Prototype v4
Parts:
- removed J1: IN, YonaFootprints:6mmStripEnd
- removed J12, J2, J3, J4, J5: MID, YonaFootprints:6mmStripMid
- removed J13: OUT, YonaFootprints:6mmStripEnd
- added J10: DAT_BRIDGE, YonaFootprints:TEDX_DAT_BRIDGE, F.Cu at (283.3, 104.8)
- added J11: DAT_BRIDGE, YonaFootprints:TEDX_DAT_BRIDGE, F.Cu at (300.0, 104.8)
- added J14: DAT_BRIDGE, YonaFootprints:TEDX_DAT_BRIDGE, F.Cu at (316.6, 104.8)
- added J15: DAT_BRIDGE, YonaFootprints:TEDX_DAT_BRIDGE, F.Cu at (333.3, 104.8)
- added J7: DAT_BRIDGE, YonaFootprints:TEDX_DAT_BRIDGE, B.Cu at (91.7, 98.2)
- added J7: DAT_BRIDGE, YonaFootprints:TEDX_DAT_BRIDGE, B.Cu at (91.7, 104.8)
- added J7: DAT_BRIDGE, YonaFootprints:TEDX_DAT_BRIDGE, B.Cu at (75.0, 98.2)
- added J7: DAT_BRIDGE, YonaFootprints:TEDX_DAT_BRIDGE, B.Cu at (75.0, 104.8)
- added J8: DAT_BRIDGE, YonaFootprints:TEDX_DAT_BRIDGE, F.Cu at (250.0, 104.8)
- added J9: DAT_BRIDGE, YonaFootprints:TEDX_DAT_BRIDGE, F.Cu at (266.7, 104.8)
- moved C12 11.3 mm to (264.1, 101.0), turned to 0 degrees
- moved C17 10.7 mm to (347.4, 99.8), turned to 0 degrees
- moved C16 10.4 mm to (330.7, 101.0), turned to 0 degrees
- moved C15 10.4 mm to (314.1, 101.0), turned to 0 degrees
- moved C13 10.4 mm to (280.7, 101.0), turned to 0 degrees
- moved C14 10.4 mm to (297.4, 101.0), turned to 0 degrees
- moved C11 3.90 mm to (252.1, 100.2), turned to 0 degrees
- moved R13 3.46 mm to (280.7, 99.5), turned to 180 degrees
- moved R16 3.46 mm to (330.7, 99.5), turned to 180 degrees
- moved R14 3.46 mm to (297.4, 99.5), turned to 180 degrees
- moved R15 3.46 mm to (314.1, 99.5), turned to 180 degrees
- moved R12 2.92 mm to (264.1, 99.5), turned to 180 degrees
- moved J10 2.50 mm to (291.7, 98.2), turned to 180 degrees
- moved J11 2.50 mm to (308.3, 98.2), turned to 180 degrees
- moved J14 2.50 mm to (325.0, 98.2), turned to 180 degrees
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Routing:
- net Net-(D14-Pad3): track 52.0 -> 73.2 mm, vias 4 -> 7
- net Net-(D15-Pad3): track 50.8 -> 71.7 mm, vias 4 -> 7
- net Net-(D13-Pad3): track 51.5 -> 72.1 mm, vias 4 -> 7
- net +5V: track 167.1 -> 149.3 mm, vias 12 -> 31
- net Net-(D12-Pad3): track 55.2 -> 72.1 mm, vias 4 -> 9
- net Net-(D16-Pad3): track 41.6 -> 55.6 mm, vias 4 -> 6
- net GND: track 167.4 -> 155.7 mm, vias 26 -> 39
- net Net-(D1-Pad6): track 43.6 -> 33.1 mm
- net Net-(D1-Pad4): track 35.8 -> 28.5 mm
- net Net-(D17-Pad3): track 12.5 -> 19.7 mm
- net Net-(C14-Pad1): track 10.5 -> 5.46 mm
- net Net-(C13-Pad1): track 10.5 -> 5.56 mm
- net Net-(C16-Pad1): track 10.5 -> 5.56 mm
- net Net-(C15-Pad1): track 10.5 -> 5.73 mm
- net Net-(C12-Pad1): track 10.2 -> 5.56 mm
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Other:
- net class Default: clearance 0.25 -> 0.1524
- rule trace_clearance: 0.25 -> 0.1524
- board text added: "NO-CONN"
- board text removed: "BIN"
- board text removed: "DIN"
- board text removed: "G"
