File: EOutside/EOutside.sch (KiCad schematic (older format))
At the start: 51 parts, among them J1 IN, J2 MID, J3 MID, J4 MID, J5 OUT, J6 PWR_BRIDGE

Commit message: Second Prototype Run
Parts:
- added J10, J11, J7, J8, J9: DAT_BRIDGE, YonaFootprints:TEDX_DAT_BRIDGE, symbol Connector:Conn_01x02_Male
Connections:
- net at D1.4 (DIN), D2.6 (BIN), J1.2 (Pin_2): now also J7.1 (Pin_1)
- net at D1.6 (BIN), J1.3 (Pin_3): now also J7.2 (Pin_2)
- net at D11.3 (DOUT), D12.4 (DIN), D13.6 (BIN)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: now also J8.2 (Pin_2)
- net at D12.3 (DOUT), D13.4 (DIN), D14.6 (BIN)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: now also J8.1 (Pin_1), J9.2 (Pin_2)
- net at D13.3 (DOUT), D14.4 (DIN), D15.6 (BIN)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: now also J10.2 (Pin_2), J9.1 (Pin_1)
- net at D14.3 (DOUT), D15.4 (DIN), J4.2 (Pin_2)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: now also J10.1 (Pin_1), J11.2 (Pin_2)
- net at D15.3 (DOUT), J5.2 (Pin_2): now also J11.1 (Pin_1)
Other:
- moved on the sheet: J6
Changed lines of the file:
@@
 	14300 4000 14300 3450
 Wire Wire Line
-	13900 4100 14300 4100
+	13900 4100 14200 4100
 Wire Wire Line
 	14050 3500 14050 3450
@@
 	15800 4000 15800 3450
 Wire Wire Line
-	15400 4100 15800 4100
+	15400 4100 15700 4100
 Wire Wire Line
 	15550 3500 15550 3450
@@
 	17300 4000 17300 3450
 Wire Wire Line
-	16900 4100 17300 4100
+	16900 4100 17200 4100
 Wire Wire Line
 	17050 3500 17050 3450
@@
 	18800 4000 18800 3450
 Wire Wire Line
-	18400 4100 18800 4100
+	18400 4100 18700 4100
 Wire Wire Line
 	18550 3500 18550 3450
@@
 L Connector:Conn_01x02_Male J6
 U 1 1 5D1D0E0E
-P 1100 5550
-F 0 "J6" H 900 5750 50  0000 C CNN
-F 1 "PWR_BRIDGE" H 1050 5650 50  0000 C CNN
-F 2 "YonaFootprints:TEDX_PWR_BRIDGE" H 1100 5550 50  0001 C CNN
-F 3 "~" H 1100 5550 50  0001 C CNN
-	1    1100 5550
+P 1250 6500
+F 0 "J6" H 1050 6700 50  0000 C CNN
+F 1 "PWR_BRIDGE" H 1200 6600 50  0000 C CNN
+F 2 "YonaFootprints:TEDX_PWR_BRIDGE" H 1250 6500 50  0001 C CNN
+F 3 "~" H 1250 6500 50  0001 C CNN
+	1    1250 6500
 	1    0    0    -1
 $EndComp
@@
 L power:+5V #PWR0101
 U 1 1 5D1D171B
-P 1400 5500
-F 0 "#PWR0101" H 1400 5350 50  0001 C CNN
-F 1 "+5V" H 1415 5673 50  0000 C CNN
-F 2 "" H 1400 5500 50  0001 C CNN
-F 3 "" H 1400 5500 50  0001 C CNN
-	1    1400 5500
+P 1550 6450
+F 0 "#PWR0101" H 1550 6300 50  0001 C CNN
+F 1 "+5V" H 1565 6623 50  0000 C CNN
+F 2 "" H 1550 6450 50  0001 C CNN
+F 3 "" H 1550 6450 50  0001 C CNN
+	1    1550 6450
 	1    0    0    -1
 $EndComp
@@
 L power:GND #PWR0102
 U 1 1 5D1D1B65
-P 1400 5700
-F 0 "#PWR0102" H 1400 5450 50  0001 C CNN
-F 1 "GND" H 1405 5527 50  0000 C CNN
-F 2 "" H 1400 5700 50  0001 C CNN
-F 3 "" H 1400 5700 50  0001 C CNN
-	1    1400 5700
-	1    0    0    -1
-$EndComp
-Wire Wire Line
-	1300 5650 1400 5650
-Wire Wire Line
-	1400 5650 1400 5700
-Wire Wire Line
-	1400 5500 1400 5550
-Wire Wire Line
-	1400 5550 1300 5550
+P 1550 6650
+F 0 "#PWR0102" H 1550 6400 50  0001 C CNN
+F 1 "GND" H 1555 6477 50  0000 C CNN
+F 2 "" H 1550 6650 50  0001 C CNN
+F 3 "" H 1550 6650 50  0001 C CNN
+	1    1550 6650
+	1    0    0    -1
+$EndComp
+Wire Wire Line
+	1450 6600 1550 6600
+Wire Wire Line
+	1550 6600 1550 6650
+Wire Wire Line
+	1550 6450 1550 6500
+Wire Wire Line
+	1550 6500 1450 6500
+$Comp
+L Connector:Conn_01x02_Male J7
+U 1 1 5CCB5ED8
+P 900 4900
+F 0 "J7" H 700 5100 50  0000 C CNN
+F 1 "DAT_BRIDGE" H 850 5000 50  0000 C CNN
+F 2 "YonaFootprints:TEDX_DAT_BRIDGE" H 900 4900 50  0001 C CNN
+F 3 "~" H 900 4900 50  0001 C CNN
+	1    900  4900
+	1    0    0    -1
+$EndComp
+Wire Wire Line
+	1200 4200 1200 5000
+Wire Wire Line
+	1200 5000 1100 5000
+Connection ~ 1200 4200
+$Comp
+L Connector:Conn_01x02_Male J9
+U 1 1 5CDE7BBE
+P 15400 5050
+F 0 "J9" H 15200 5250 50  0000 C CNN
+F 1 "DAT_BRIDGE" H 15350 5150 50  0000 C CNN
+F 2 "YonaFootprints:TEDX_DAT_BRIDGE" H 15400 5050 50  0001 C CNN
+F 3 "~" H 15400 5050 50  0001 C CNN
+	1    15400 5050
+	1    0    0    -1
+$EndComp
+Wire Wire Line
+	15700 4100 15700 5050
+Wire Wire Line
+	15700 5050 15600 5050
+Connection ~ 15700 4100
+Wire Wire Line
+	15700 4100 15800 4100
+Wire Wire Line
+	15650 4450 15650 5150
+Wire Wire Line
+	15650 5150 15600 5150
+Connection ~ 15650 4450
+$Comp
+L Connector:Conn_01x02_Male J10
+U 1 1 5CE1C94C
+P 16900 5050
+F 0 "J10" H 16700 5250 50  0000 C CNN
+F 1 "DAT_BRIDGE" H 16850 5150 50  0000 C CNN
+F 2 "YonaFootprints:TEDX_DAT_BRIDGE" H 16900 5050 50  0001 C CNN
+F 3 "~" H 16900 5050 50  0001 C CNN
+	1    16900 5050
+	1    0    0    -1
+$EndComp
+$Comp
+L Connector:Conn_01x02_Male J11
+U 1 1 5CE2E5E6
+P 18400 5050
+F 0 "J11" H 18200 5250 50  0000 C CNN
+F 1 "DAT_BRIDGE" H 18350 5150 50  0000 C CNN
+F 2 "YonaFootprints:TEDX_DAT_BRIDGE" H 18400 5050 50  0001 C CNN
+F 3 "~" H 18400 5050 50  0001 C CNN
+	1    18400 5050
+	1    0    0    -1
+$EndComp
+Wire Wire Line
+	17100 5050 17200 5050
+Wire Wire Line
+	17200 5050 17200 4100
+Connection ~ 17200 4100
+Wire Wire Line
+	17200 4100 17300 4100
+Wire Wire Line
+	17150 4450 17150 5150
+Wire Wire Line
+	17150 5150 17100 5150
+Connection ~ 17150 4450
+Wire Wire Line
+	18700 4100 18700 5050
+Wire Wire Line
+	18700 5050 18600 5050
+Connection ~ 18700 4100
+Wire Wire Line
+	18700 4100 18800 4100
+Wire Wire Line
+	18650 4450 18650 5150
+Wire Wire Line
+	18650 5150 18600 5150
+Connection ~ 18650 4450
+$Comp
+L Connector:Conn_01x02_Male J8
+U 1 1 5CE8A8C0
+P 13900 5050
+F 0 "J8" H 13700 5250 50  0000 C CNN
+F 1 "DAT_BRIDGE" H 13850 5150 50  0000 C CNN
+F 2 "YonaFootprints:TEDX_DAT_BRIDGE" H 13900 5050 50  0001 C CNN
+F 3 "~" H 13900 5050 50  0001 C CNN
+	1    13900 5050
+	1    0    0    -1
+$EndComp
+Wire Wire Line
+	14100 5050 14200 5050
+Wire Wire Line
+	14200 5050 14200 4100
+Connection ~ 14200 4100
+Wire Wire Line
+	14200 4100 14300 4100
+Wire Wire Line
+	14150 4450 14150 5150
+Wire Wire Line
+	14150 5150 14100 5150
+Connection ~ 14150 4450
+Wire Wire Line
+	1150 4450 1150 4900
+Wire Wire Line
+	1150 4900 1100 4900
+Connection ~ 1150 4450
 $EndSCHEMATC

Commit message: Before changing Outside Struts to not have connectors
Parts:
- added C16, C17: .1uF, Capacitor_SMD:C_0603_1608Metric, symbol Device:C
- added D16, D17: WS2813, LED_SMD:LED_WS2812_PLCC6_5.0x5.0mm_P1.6mm, symbol LED:WS2813
- added J12: MID, YonaFootprints:6mmStripMid, symbol Connector:Conn_01x04_Female
- added J13: OUT, YonaFootprints:6mmStripEnd, symbol Connector:Conn_01x04_Female
- added J14, J15: DAT_BRIDGE, YonaFootprints:TEDX_DAT_BRIDGE, symbol Connector:Conn_01x02_Male
- added R16, R17: 330, Resistor_SMD:R_0603_1608Metric, symbol Device:R
- J5: value OUT -> MID; footprint YonaFootprints:6mmStripEnd -> YonaFootprints:6mmStripMid
Connections:
- net +5V: now also D16.2 (VDD), D17.2 (VDD), J12.1 (Pin_1), J13.1 (Pin_1), R16.1, R17.1
- net GND: now also C16.2, C17.2, D16.5 (GND), D17.5 (GND), J12.4 (Pin_4), J13.4 (Pin_4)
- net at D14.3 (DOUT), D15.4 (DIN), J10.1 (Pin_1)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: now also D16.6 (BIN)
- net at D15.3 (DOUT), J11.1 (Pin_1), J5.2 (Pin_2): now also D16.4 (DIN), D17.6 (BIN), J12.3 (Pin_3), J14.2 (Pin_2)
- new net: D16.3 (DOUT), D17.4 (DIN), J12.2 (Pin_2), J13.3 (Pin_3), J14.1 (Pin_1), J15.2 (Pin_2)
- new net: C16.1, D16.1 (VCC), R16.2
- new net: D17.3 (DOUT), J13.2 (Pin_2), J15.1 (Pin_1)
- new net: C17.1, D17.1 (VCC), R17.2

Commit message: Prototype v4
Parts:
- removed J1: IN, YonaFootprints:6mmStripEnd, symbol Connector:Conn_01x04_Male
- removed J12, J2, J3, J4, J5: MID, YonaFootprints:6mmStripMid, symbol Connector:Conn_01x04_Female
- removed J13: OUT, YonaFootprints:6mmStripEnd, symbol Connector:Conn_01x04_Female
Changed lines of the file:
@@
 E Strut\n17 LEDs\nx3
-$Comp
-L Connector:Conn_01x04_Male J1
-U 1 1 5CCD490D
-P 900 4100
-F 0 "J1" H 1008 4381 50  0000 C CNN
-F 1 "IN" H 1008 4290 50  0000 C CNN
-F 2 "YonaFootprints:6mmStripEnd" H 900 4100 50  0001 C CNN
-F 3 "~" H 900 4100 50  0001 C CNN
-	1    900  4100
-	1    0    0    -1
-$EndComp
 $Comp
 L Device:C C1
@@
 $EndComp
 Connection ~ 1950 4500
-Wire Wire Line
-	1100 4500 1100 4300
-Wire Wire Line
-	1100 4500 1500 4500
-Wire Wire Line
-	1100 4000 1100 3450
-Wire Wire Line
-	1100 3450 1400 3450
 Connection ~ 1400 3450
 Wire Wire Line
-	1100 4100 1150 4100
-Connection ~ 1150 4100
-Wire Wire Line
 	1150 4100 1200 4100
-Wire Wire Line
-	1100 4200 1200 4200
 Wire Wire Line
 	1400 3450 1950 3450
@@
 	14250 4300 14250 4500
 $Comp
-L Connector:Conn_01x04_Female J2
-U 1 1 5CE3CD62
-P 14500 4100
-F 0 "J2" H 14350 4300 50  0000 L CNN
-F 1 "MID" H 14350 3800 50  0000 L CNN
-F 2 "YonaFootprints:6mmStripMid" H 14500 4100 50  0001 C CNN
-F 3 "~" H 14500 4100 50  0001 C CNN
-	1    14500 4100
-	1    0    0    -1
-$EndComp
-$Comp
 L Device:R R12
 U 1 1 5CE3CD68
@@
 	1    0    0    -1
 $EndComp
-Wire Wire Line
-	14250 4300 14300 4300
-Wire Wire Line
-	14150 4200 14300 4200
 Connection ~ 13600 4500
 Wire Wire Line
@@
 	15750 4300 15750 4500
 $Comp
-L Connector:Conn_01x04_Female J3
-U 1 1 5CEE64A9
-P 16000 4100
-F 0 "J3" H 15850 4300 50  0000 L CNN
-F 1 "MID" H 15850 3800 50  0000 L CNN
-F 2 "YonaFootprints:6mmStripMid" H 16000 4100 50  0001 C CNN
-F 3 "~" H 16000 4100 50  0001 C CNN
-	1    16000 4100
-	1    0    0    -1
-$EndComp
-$Comp
 L Device:R R13
 U 1 1 5CEE64AF
@@
 	1    0    0    -1
 $EndComp
-Wire Wire Line
-	15750 4300 15800 4300
-Wire Wire Line
-	15650 4200 15800 4200
 Connection ~ 15100 4500
 Wire Wire Line
@@
 	17250 4300 17250 4500
 $Comp
-L Connector:Conn_01x04_Female J4
-U 1 1 5CEF1C79
-P 17500 4100
-F 0 "J4" H 17350 4300 50  0000 L CNN
-F 1 "MID" H 17350 3800 50  0000 L CNN
-F 2 "YonaFootprints:6mmStripMid" H 17500 4100 50  0001 C CNN
-F 3 "~" H 17500 4100 50  0001 C CNN
-	1    17500 4100
-	1    0    0    -1
-$EndComp
-$Comp
 L Device:R R14
 U 1 1 5CEF1C7F
@@
 	1    0    0    -1
 $EndComp
-Wire Wire Line
-	17250 4300 17300 4300
-Wire Wire Line
-	17150 4200 17300 4200
 Connection ~ 16600 4500
 Wire Wire Line
@@
 	18750 4300 18750 4500
 $Comp
-L Connector:Conn_01x04_Female J5
-U 1 1 5CF01720
-P 19000 4100
-F 0 "J5" H 18850 4300 50  0000 L CNN
-F 1 "MID" H 18850 3800 50  0000 L CNN
-F 2 "YonaFootprints:6mmStripMid" H 19000 4100 50  0001 C CNN
-F 3 "~" H 19000 4100 50  0001 C CNN
-	1    19000 4100
-	1    0    0    -1
-$EndComp
-$Comp
 L Device:R R15
 U 1 1 5CF01726
@@
 Wire Wire Line
 	14300 4000 14700 4000
-Connection ~ 14300 4000
-Connection ~ 14300 4100
-Wire Wire Line
-	14300 4200 14800 4200
-Connection ~ 14300 4200
-Wire Wire Line
-	14700 4300 14300 4300
-Connection ~ 14300 4300
-Wire Wire Line
-	14300 4100 14750 4100
 Wire Wire Line
 	15800 4000 16200 4000
-Connection ~ 15800 4000
-Wire Wire Line
-	15800 4100 16250 4100
-Connection ~ 15800 4100
-Wire Wire Line
-	15800 4200 16300 4200
-Connection ~ 15800 4200
-Wire Wire Line
-	16200 4300 15800 4300
-Connection ~ 15800 4300
 Wire Wire Line
 	17300 4000 17700 4000
-Connection ~ 17300 4000
-Wire Wire Line
-	17300 4100 17750 4100
-Connection ~ 17300 4100
-Wire Wire Line
-	17300 4200 17800 4200
-Connection ~ 17300 4200
-Wire Wire Line
-	17300 4300 17700 4300
-Connection ~ 17300 4300
 $Comp
 L Connector:Conn_01x02_Male J6
@@
 Wire Wire Line
 	1200 5000 1100 5000
-Connection ~ 1200 4200
 $Comp
 L Connector:Conn_01x02_Male J9
@@
 Connection ~ 15700 4100
 Wire Wire Line
-	15700 4100 15800 4100
-Wire Wire Line
 	15650 4450 15650 5150
 Wire Wire Line
@@
 Connection ~ 17200 4100
 Wire Wire Line
-	17200 4100 17300 4100
-Wire Wire Line
 	17150 4450 17150 5150
 Wire Wire Line
@@
 Connection ~ 14200 4100
 Wire Wire Line
-	14200 4100 14300 4100
-Wire Wire Line
 	14150 4450 14150 5150
 Wire Wire Line
@@
 Wire Wire Line
 	20250 4300 20250 4500
-$Comp
-L Connector:Conn_01x04_Female J12
-U 1 1 5CD2718F
-P 20500 4100
-F 0 "J12" H 20350 4300 50  0000 L CNN
-F 1 "MID" H 20350 3800 50  0000 L CNN
-F 2 "YonaFootprints:6mmStripMid" H 20500 4100 50  0001 C CNN
-F 3 "~" H 20500 4100 50  0001 C CNN
-	1    20500 4100
-	1    0    0    -1
-$EndComp
 $Comp
 L Device:R R16
@@
 Wire Wire Line
 	20700 4500 20700 4300
-Connection ~ 21550 4500
-Wire Wire Line
-	21750 4500 21550 4500
-Wire Wire Line
-	21750 4300 21750 4500
-$Comp
-L Connector:Conn_01x04_Female J13
-U 1 1 5CD41C1D
-P 22000 4100
-F 0 "J13" H 21850 4300 50  0000 L CNN
-F 1 "OUT" H 21850 3800 50  0000 L CNN
-F 2 "YonaFootprints:6mmStripEnd" H 22000 4100 50  0001 C CNN
-F 3 "~" H 22000 4100 50  0001 C CNN
-	1    22000 4100
-	1    0    0    -1
-$EndComp
 $Comp
 L Device:R R17
@@
 Connection ~ 21550 3800
 Wire Wire Line
-	21800 4000 21800 3450
-Wire Wire Line
 	21400 4100 21700 4100
 Wire Wire Line
 	21550 3500 21550 3450
-Connection ~ 21550 3450
-Wire Wire Line
-	21550 3450 21800 3450
 Wire Wire Line
 	21000 3800 21000 3450
@@
 	1    0    0    -1
 $EndComp
-Wire Wire Line
-	21750 4300 21800 4300
-Wire Wire Line
-	21650 4200 21800 4200
 Connection ~ 21100 4500
 Wire Wire Line
@@
 Wire Wire Line
 	20750 4450 21650 4450
-Wire Wire Line
-	21650 4200 21650 4450
 $Comp
 L Device:C C17
@@
 Wire Wire Line
 	21700 5050 21600 5050
-Connection ~ 21700 4100
-Wire Wire Line
-	21700 4100 21800 4100
 Wire Wire Line
 	21650 4450 21650 5150
 Wire Wire Line
 	21650 5150 21600 5150
-Connection ~ 21650 4450
+Wire Wire Line
+	14200 4100 14750 4100
+Wire Wire Line
+	14150 4200 14800 4200
+Wire Wire Line
+	14250 4300 14700 4300
+Wire Wire Line
+	15700 4100 16250 4100
+Wire Wire Line
+	15650 4200 16300 4200
+Wire Wire Line
+	15750 4300 16200 4300
+Wire Wire Line
+	17200 4100 17750 4100
+Wire Wire Line
+	17150 4200 17800 4200
+Wire Wire Line
+	17250 4300 17700 4300
 $EndSCHEMATC
