File: FInside/Strut.kicad_pcb (KiCad board)
At the start: 4 copper layers, 309.6 x 138.1 mm, 53 parts, among them J1 IN, J2 OUT

Commit message: First iteration of all struts
Parts:
- removed C17: 100NF, Capacitor_SMD:C_0805_2012Metric
- removed D17: WS2813, LED_SMD:LED_WS2812_PLCC6_5.0x5.0mm_P1.6mm
- removed R17: 330, Resistor_SMD:R_0805_2012Metric
- moved J2 43.5 mm to (326.9, 185.2)
- moved R16 39.8 mm to (320.4, 183.3)
- moved R9 39.7 mm to (204.5, 183.4), turned to 180 degrees
- moved C10 39.5 mm to (227.7, 188.1)
- moved C11 39.5 mm to (244.4, 188.1)
- moved C12 39.5 mm to (261.5, 188.1)
- moved C13 39.5 mm to (278.1, 188.1)
- moved C14 39.5 mm to (294.8, 188.1)
- moved C2 39.5 mm to (94.5, 188.1)
- moved C3 39.5 mm to (111.2, 188.1)
- moved C4 39.5 mm to (127.8, 188.1)
- moved C5 39.5 mm to (144.5, 188.1)
- moved C6 39.5 mm to (161.1, 188.1)
- moved C7 39.5 mm to (177.8, 188.1)
- moved C8 39.5 mm to (194.4, 188.1)
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Connections:
- J2 pad 2: Net-(D17-Pad3) -> Net-(D16-Pad3)
Routing:
- net Net-(D15-Pad3): track 36.1 -> 13.0 mm
- net Net-(C17-Pad1): track 11.8 -> 0.00 mm
- net +5V: track 89.0 -> 78.9 mm
- net Net-(D17-Pad3): track 9.86 -> 0.00 mm, vias 1 -> 0
- net Net-(D16-Pad3): track 13.5 -> 5.31 mm
- net GND: track 101.3 -> 93.8 mm, vias 20 -> 19
- net Net-(C1-Pad1): track 15.6 -> 10.3 mm
- net Net-(D1-Pad4): track 33.8 -> 28.6 mm
- net Net-(D10-Pad6): track 36.8 -> 33.0 mm
- net Net-(C15-Pad1): track 6.15 -> 9.50 mm
- net Net-(C16-Pad1): track 12.3 -> 10.4 mm
- net Net-(C9-Pad1): track 9.89 -> 9.22 mm, vias 2 -> 0
Other:
- outline, holes or cut-outs redrawn
