File: FInside/FInside.kicad_pcb (KiCad board)
At the start: 2 copper layers, 279.7 x 14.3 mm, 64 parts, among them J1 IN, J2 IN2, J3 OUT2, J4 PWR_BRIDGE, J5 OUT

Commit message: Second Prototype Run
Parts:
- removed J3: OUT2, YonaFootprints:TEDX_IN2
- removed the J4 at (102.9, 142.2)
- removed the J4 at (169.6, 142.2)
- removed the J4 at (152.8, 142.2)
- removed the J4 at (119.6, 142.2)
- removed the J4 at (136.3, 142.2)
- removed the J4 at (269.6, 142.2)
- removed the J4 at (252.9, 142.2)
- removed the J4 at (236.3, 142.2)
- removed the J4 at (219.6, 142.2)
- removed the J4 at (202.9, 142.2)
- removed the J4 at (186.3, 142.2)
- removed JP1: DOUT2_ENABLE, Jumper:SolderJumper-2_P1.3mm_Open_TrianglePad1.0x1.5mm
- removed JP2: BOUT2_ENABLE, Jumper:SolderJumper-2_P1.3mm_Open_TrianglePad1.0x1.5mm
- added J4: PWR_BRIDGE, YonaFootprints:TEDX_PWR_BRIDGE_TALL, B.Cu at (252.9, 145.0)
- added J4: PWR_BRIDGE, YonaFootprints:TEDX_PWR_BRIDGE_TALL, B.Cu at (136.3, 145.0)
- added J6: DAT_BRIDGE, YonaFootprints:TEDX_DAT_BRIDGE_TALL, B.Cu at (286.3, 145.0)
Routing:
- net Net-(J3-Pad1): track 264.6 -> 0.00 mm, vias 4 -> 0
- net Net-(J3-Pad2): track 260.1 -> 0.00 mm, vias 4 -> 0
- net +5V: track 140.6 -> 67.4 mm, vias 35 -> 16
- net GND: track 138.3 -> 71.8 mm
- net /DOUT: track 16.0 -> 28.8 mm, vias 1 -> 4
- net /BOUT: track 37.6 -> 42.0 mm
- net /DIN: track 32.6 -> 30.4 mm
- net Net-(C1-Pad1): track 10.7 -> 12.4 mm
- net Net-(D5-Pad3): track 32.1 -> 33.6 mm
- net Net-(D6-Pad3): track 32.0 -> 33.4 mm
- net Net-(D3-Pad3): track 31.9 -> 33.2 mm
- net Net-(D10-Pad6): track 31.9 -> 33.2 mm
- net Net-(D10-Pad4): track 31.9 -> 33.1 mm
- net Net-(D7-Pad3): track 32.0 -> 33.2 mm
- net Net-(D11-Pad3): track 31.7 -> 33.0 mm
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Other:
- board text removed: "BK-OUT C/O ENABLE"
- board text removed: "DAT-OUT C/O ENABLE"

Commit message: Before changing Outside Struts to not have connectors
Routing:
- net Net-(D1-Pad3): track 35.0 -> 32.6 mm, vias 0 -> 2
- net Net-(D6-Pad3): track 33.4 -> 31.2 mm, vias 2 -> 4
- net Net-(D5-Pad3): track 33.6 -> 31.5 mm, vias 2 -> 4
- net Net-(D7-Pad3): track 33.2 -> 31.1 mm, vias 2 -> 4
- net Net-(D2-Pad3): track 33.4 -> 31.3 mm, vias 2 -> 4
- net Net-(D3-Pad3): track 33.2 -> 31.1 mm, vias 2 -> 4
- net /BOUT: track 42.0 -> 40.0 mm, vias 1 -> 3
- net Net-(D10-Pad3): track 33.0 -> 31.0 mm, vias 2 -> 4
- net Net-(D10-Pad4): track 33.1 -> 31.2 mm, vias 2 -> 4
- net Net-(D10-Pad6): track 33.2 -> 31.2 mm, vias 2 -> 4
- net Net-(J2-Pad1): track 262.2 -> 260.5 mm, vias 5 -> 4
- net Net-(D4-Pad3): track 33.1 -> 31.5 mm, vias 2 -> 4
- net Net-(D11-Pad3): track 33.0 -> 31.5 mm, vias 2 -> 4
- net /DIN: track 30.4 -> 28.9 mm, vias 0 -> 2
- net Net-(D13-Pad3): track 34.1 -> 32.7 mm, vias 2 -> 4
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
Commit message: Prototype v4
Parts:
- removed the J2 at (315.4, 148.2)
- added J2: PWR_BRIDGE2, YonaFootprints:TEDX_PWR_BRIDGE, B.Cu at (236.3, 152.1)
- added J2: PWR_BRIDGE2, YonaFootprints:TEDX_PWR_BRIDGE, B.Cu at (119.6, 152.1)
- added REF**: TEDX_DAT_BRIDGE, YonaFootprints:TEDX_DAT_BRIDGE, B.Cu at (86.3, 152.1)
- JP3: value DOUT2_ENABLE -> CO_DIN_ENABLE; moved to F.Cu
- JP4: value BOUT2_ENABLE -> CO_BIN_ENABLE; moved to F.Cu
- moved JP4 21.2 mm to (54.8, 148.1)
- moved JP3 9.31 mm to (54.8, 145.5)
Connections:
- J5 pad 2: /DOUT -> /CO_DIN
- J5 pad 3: /BOUT -> /CO_BIN
- JP3 pad 1: /DIN -> /CO_DIN
- JP3 pad 2: Net-(J2-Pad1) -> /DIN
- JP4 pad 1: /BIN -> /CO_BIN
- JP4 pad 2: Net-(J2-Pad2) -> /BIN
Routing:
- net /CO_BIN: track 0.00 -> 281.6 mm, vias 0 -> 5
- net /CO_DIN: track 0.00 -> 272.8 mm, vias 0 -> 5
- net Net-(J2-Pad1): track 260.5 -> 0.00 mm, vias 4 -> 0
- net Net-(J2-Pad2): track 254.2 -> 0.00 mm, vias 4 -> 0
- net /BOUT: track 40.0 -> 27.4 mm, vias 3 -> 1
- net +5V: track 66.2 -> 76.4 mm, vias 16 -> 20
- net /BIN: track 19.3 -> 12.3 mm, vias 2 -> 0
- net /DOUT: track 30.1 -> 23.1 mm, vias 4 -> 3
- net GND: track 72.1 -> 78.3 mm, vias 31 -> 33
- net Net-(D1-Pad3): track 32.6 -> 30.6 mm, vias 2 -> 4
- net /DIN: track 28.9 -> 30.1 mm
Other:
- board text added: "BO"
- board text added: "C/O BIN"
- board text added: "C/O DIN"
- board text added: "C/O ENABLE"
- board text added: "DO"
- board text added: "G"
- board text added: "NO-CONN"
- board text removed: "BK-IN C/O ENABLE"
- board text removed: "DAT-IN C/O ENABLE"
