File: FInside/FInside.sch (KiCad schematic (older format))
At the start: 54 parts, among them J1 IN, J2 IN2, J3 OUT2, J4 PWR_BRIDGE, J5 OUT

Commit message: Second Prototype Run
Parts:
- removed J3: OUT2, YonaFootprints:TEDX_IN2, symbol Connector:Conn_01x02_Female
- removed JP1: DOUT2_ENABLE, Jumper:SolderJumper-2_P1.3mm_Open_TrianglePad1.0x1.5mm, symbol Jumper:Jumper_2_Open
- removed JP2: BOUT2_ENABLE, Jumper:SolderJumper-2_P1.3mm_Open_TrianglePad1.0x1.5mm, symbol Jumper:Jumper_2_Open
- added J6: DAT_BRIDGE, YonaFootprints:TEDX_DAT_BRIDGE_TALL, symbol Connector:Conn_01x02_Male
Connections:
- net BOUT: now also J6.2 (Pin_2)
- net DOUT: now also J6.1 (Pin_1)
Other:
- moved on the sheet: J4
Changed lines of the file:
@@
 Text Label 18550 4100 2    50   ~ 0
 BOUT
-$Comp
-L Connector:Conn_01x02_Female J3
-U 1 1 5CF8C196
-P 19500 4550
-F 0 "J3" H 19528 4526 50  0000 L CNN
-F 1 "OUT2" H 19528 4435 50  0000 L CNN
-F 2 "YonaFootprints:TEDX_IN2" H 19500 4550 50  0001 C CNN
-F 3 "~" H 19500 4550 50  0001 C CNN
-	1    19500 4550
-	1    0    0    -1
-$EndComp
-Wire Wire Line
-	18350 4100 18350 4650
 Wire Wire Line
 	18350 4100 18550 4100
-Wire Wire Line
-	18400 4000 18400 4550
-$Comp
-L Jumper:Jumper_2_Open JP1
-U 1 1 5CFBB150
-P 19100 4550
-F 0 "JP1" H 19100 4785 50  0000 C CNN
-F 1 "DOUT2_ENABLE" H 19100 4694 50  0000 C CNN
-F 2 "Jumper:SolderJumper-2_P1.3mm_Open_TrianglePad1.0x1.5mm" H 19100 4550 50  0001 C CNN
-F 3 "~" H 19100 4550 50  0001 C CNN
-	1    19100 4550
-	1    0    0    -1
-$EndComp
-$Comp
-L Jumper:Jumper_2_Open JP2
-U 1 1 5CFBCECE
-P 19100 4650
-F 0 "JP2" H 19100 4500 50  0000 C CNN
-F 1 "BOUT2_ENABLE" H 19100 4400 50  0000 C CNN
-F 2 "Jumper:SolderJumper-2_P1.3mm_Open_TrianglePad1.0x1.5mm" H 19100 4650 50  0001 C CNN
-F 3 "~" H 19100 4650 50  0001 C CNN
-	1    19100 4650
-	1    0    0    -1
-$EndComp
-Wire Wire Line
-	18400 4550 18900 4550
-Wire Wire Line
-	18350 4650 18900 4650
 $Comp
 L Jumper:Jumper_2_Open JP3
@@
 L Connector:Conn_01x02_Male J4
 U 1 1 5CD3CF2F
-P 17700 5200
-F 0 "J4" H 17650 5400 50  0000 C CNN
-F 1 "PWR_BRIDGE" H 17600 5300 50  0000 C CNN
-F 2 "YonaFootprints:TEDX_PWR_BRIDGE_TALL" H 17700 5200 50  0001 C CNN
-F 3 "~" H 17700 5200 50  0001 C CNN
-	1    17700 5200
+P 16900 5450
+F 0 "J4" H 16850 5650 50  0000 C CNN
+F 1 "PWR_BRIDGE" H 16800 5550 50  0000 C CNN
+F 2 "YonaFootprints:TEDX_PWR_BRIDGE_TALL" H 16900 5450 50  0001 C CNN
+F 3 "~" H 16900 5450 50  0001 C CNN
+	1    16900 5450
 	1    0    0    -1
 $EndComp
@@
 L power:+5V #PWR0125
 U 1 1 5CD3DA97
-P 17900 5200
-F 0 "#PWR0125" H 17900 5050 50  0001 C CNN
-F 1 "+5V" H 17915 5373 50  0000 C CNN
-F 2 "" H 17900 5200 50  0001 C CNN
-F 3 "" H 17900 5200 50  0001 C CNN
-	1    17900 5200
+P 17100 5450
+F 0 "#PWR0125" H 17100 5300 50  0001 C CNN
+F 1 "+5V" H 17115 5623 50  0000 C CNN
+F 2 "" H 17100 5450 50  0001 C CNN
+F 3 "" H 17100 5450 50  0001 C CNN
+	1    17100 5450
 	1    0    0    -1
 $EndComp
@@
 L power:GND #PWR0126
 U 1 1 5CD3DFDA
-P 17900 5300
-F 0 "#PWR0126" H 17900 5050 50  0001 C CNN
-F 1 "GND" H 17905 5127 50  0000 C CNN
-F 2 "" H 17900 5300 50  0001 C CNN
-F 3 "" H 17900 5300 50  0001 C CNN
-	1    17900 5300
+P 17100 5550
+F 0 "#PWR0126" H 17100 5300 50  0001 C CNN
+F 1 "GND" H 17105 5377 50  0000 C CNN
+F 2 "" H 17100 5550 50  0001 C CNN
+F 3 "" H 17100 5550 50  0001 C CNN
+	1    17100 5550
 	1    0    0    -1
 $EndComp
+$Comp
+L Connector:Conn_01x02_Male J6
+U 1 1 5D019AB8
+P 18100 5150
+F 0 "J6" H 18208 5331 50  0000 C CNN
+F 1 "DAT_BRIDGE" H 18208 5240 50  0000 C CNN
+F 2 "YonaFootprints:TEDX_DAT_BRIDGE_TALL" H 18100 5150 50  0001 C CNN
+F 3 "~" H 18100 5150 50  0001 C CNN
+	1    18100 5150
+	1    0    0    -1
+$EndComp
+Wire Wire Line
+	18400 5150 18300 5150
+Wire Wire Line
+	18350 5250 18300 5250
+Wire Wire Line
+	18400 4000 18400 5150
+Wire Wire Line
+	18350 4100 18350 5250
 $EndSCHEMATC

Commit message: Prototype v4
Parts:
- J2: value IN2 -> PWR_BRIDGE2; footprint YonaFootprints:TEDX_IN2 -> YonaFootprints:TEDX_PWR_BRIDGE
- JP3: value DOUT2_ENABLE -> CO_DIN_ENABLE
- JP4: value BOUT2_ENABLE -> CO_BIN_ENABLE
Connections:
- net +5V: now also J2.1 (Pin_1)
- net BIN: now also JP4.2 (B); no longer JP4.1 (A)
- net BOUT: no longer J5.3 (Pin_3)
- net DIN: now also JP3.2 (B); no longer JP3.1 (A)
- net DOUT: no longer J5.2 (Pin_2)
- net GND: now also J2.2 (Pin_2)
- new net CO_BIN: J5.3 (Pin_3), JP4.1 (A)
- new net CO_DIN: J5.2 (Pin_2), JP3.1 (A)
Other:
- moved on the sheet: J5, J6, JP3, JP4
Changed lines of the file:
@@
 L Connector:Conn_01x04_Female J5
 U 1 1 5CF01720
-P 18750 4000
-F 0 "J5" H 18600 4200 50  0000 L CNN
-F 1 "OUT" H 18600 3700 50  0000 L CNN
-F 2 "YonaFootprints:TEDX_INNER_4" H 18750 4000 50  0001 C CNN
-F 3 "~" H 18750 4000 50  0001 C CNN
-	1    18750 4000
+P 19200 4000
+F 0 "J5" H 19050 4200 50  0000 L CNN
+F 1 "OUT" H 19050 3700 50  0000 L CNN
+F 2 "YonaFootprints:TEDX_INNER_4" H 19200 4000 50  0001 C CNN
+F 3 "~" H 19200 4000 50  0001 C CNN
+	1    19200 4000
 	1    0    0    -1
 $EndComp
@@
 Wire Wire Line
 	17300 4350 18200 4350
-Wire Wire Line
-	18200 4100 18200 4350
 $Comp
 L Device:C C15
@@
 	17000 4400 17650 4400
 Wire Wire Line
-	18550 4000 18400 4000
-Wire Wire Line
-	18550 4200 18450 4200
-Wire Wire Line
-	18450 4200 18450 4400
-Wire Wire Line
-	18550 3350 18550 3900
-$Comp
-L Connector:Conn_01x02_Male J2
-U 1 1 5CEC36A1
-P 950 4800
-F 0 "J2" H 1058 4981 50  0000 C CNN
-F 1 "IN2" H 1058 4890 50  0000 C CNN
-F 2 "YonaFootprints:TEDX_IN2" H 950 4800 50  0001 C CNN
-F 3 "~" H 950 4800 50  0001 C CNN
-	1    950  4800
-	1    0    0    -1
-$EndComp
-Wire Wire Line
-	1700 4800 1900 4800
-Wire Wire Line
 	1900 4800 1900 4350
 Connection ~ 1900 4350
-Wire Wire Line
-	1950 4100 1950 4900
-Wire Wire Line
-	1950 4900 1700 4900
 Connection ~ 1950 4100
 Wire Wire Line
@@
 Text Label 1550 4100 0    50   ~ 0
 BIN
-Text Label 18550 4000 2    50   ~ 0
+Text Label 17850 5150 0    50   ~ 0
 DOUT
-Text Label 18550 4100 2    50   ~ 0
+Text Label 17850 5250 0    50   ~ 0
 BOUT
-Wire Wire Line
-	18350 4100 18550 4100
 $Comp
 L Jumper:Jumper_2_Open JP3
 U 1 1 5CFF526D
-P 1500 4800
-F 0 "JP3" H 1500 5035 50  0000 C CNN
-F 1 "DOUT2_ENABLE" H 1500 4944 50  0000 C CNN
-F 2 "Jumper:SolderJumper-2_P1.3mm_Open_TrianglePad1.0x1.5mm" H 1500 4800 50  0001 C CNN
-F 3 "~" H 1500 4800 50  0001 C CNN
-	1    1500 4800
+P 2700 4800
+F 0 "JP3" H 2700 5035 50  0000 C CNN
+F 1 "CO_DIN_ENABLE" H 2700 4944 50  0000 C CNN
+F 2 "Jumper:SolderJumper-2_P1.3mm_Open_TrianglePad1.0x1.5mm" H 2700 4800 50  0001 C CNN
+F 3 "~" H 2700 4800 50  0001 C CNN
+	1    2700 4800
 	-1   0    0    -1
 $EndComp
@@
 L Jumper:Jumper_2_Open JP4
 U 1 1 5CFF5273
-P 1500 4900
-F 0 "JP4" H 1500 4750 50  0000 C CNN
-F 1 "BOUT2_ENABLE" H 1500 4650 50  0000 C CNN
-F 2 "Jumper:SolderJumper-2_P1.3mm_Open_TrianglePad1.0x1.5mm" H 1500 4900 50  0001 C CNN
-F 3 "~" H 1500 4900 50  0001 C CNN
-	1    1500 4900
+P 2700 4900
+F 0 "JP4" H 2700 4750 50  0000 C CNN
+F 1 "CO_BIN_ENABLE" H 2700 4650 50  0000 C CNN
+F 2 "Jumper:SolderJumper-2_P1.3mm_Open_TrianglePad1.0x1.5mm" H 2700 4900 50  0001 C CNN
+F 3 "~" H 2700 4900 50  0001 C CNN
+	1    2700 4900
 	-1   0    0    -1
 $EndComp
@@
 Connection ~ 17000 3350
 Connection ~ 17000 4400
-Wire Wire Line
-	1300 4800 1150 4800
-Wire Wire Line
-	1150 4900 1300 4900
-Wire Wire Line
-	18200 4100 18350 4100
-Connection ~ 18350 4100
-Wire Wire Line
-	17950 4000 18400 4000
-Connection ~ 18400 4000
-Wire Wire Line
-	18550 3350 18100 3350
 Connection ~ 18100 3350
-Wire Wire Line
-	18100 4400 18450 4400
 Connection ~ 18100 4400
 $Comp
@@
 L Connector:Conn_01x02_Male J6
 U 1 1 5D019AB8
-P 18100 5150
-F 0 "J6" H 18208 5331 50  0000 C CNN
-F 1 "DAT_BRIDGE" H 18208 5240 50  0000 C CNN
-F 2 "YonaFootprints:TEDX_DAT_BRIDGE_TALL" H 18100 5150 50  0001 C CNN
-F 3 "~" H 18100 5150 50  0001 C CNN
-	1    18100 5150
-	1    0    0    -1
-$EndComp
-Wire Wire Line
-	18400 5150 18300 5150
-Wire Wire Line
-	18350 5250 18300 5250
-Wire Wire Line
-	18400 4000 18400 5150
-Wire Wire Line
-	18350 4100 18350 5250
+P 17650 5150
+F 0 "J6" H 17700 5400 50  0000 C CNN
+F 1 "DAT_BRIDGE" H 17850 5300 50  0000 C CNN
+F 2 "YonaFootprints:TEDX_DAT_BRIDGE_TALL" H 17650 5150 50  0001 C CNN
+F 3 "~" H 17650 5150 50  0001 C CNN
+	1    17650 5150
+	1    0    0    -1
+$EndComp
+Wire Wire Line
+	18200 4350 18200 5250
+Wire Wire Line
+	17850 5250 18200 5250
+Wire Wire Line
+	17950 4000 18250 4000
+Wire Wire Line
+	18250 4000 18250 5150
+Wire Wire Line
+	17850 5150 18250 5150
+Wire Wire Line
+	2500 4900 1950 4900
+Text Label 3250 4800 2    50   ~ 0
+CO_DIN
+Text Label 3250 4900 2    50   ~ 0
+CO_BIN
+Wire Wire Line
+	3250 4900 2900 4900
+Wire Wire Line
+	2900 4800 3250 4800
+Text Label 18650 4000 0    50   ~ 0
+CO_DIN
+Text Label 18650 4100 0    50   ~ 0
+CO_BIN
+Wire Wire Line
+	18650 4000 19000 4000
+Wire Wire Line
+	19000 4100 18650 4100
+Wire Wire Line
+	19000 3900 19000 3350
+Wire Wire Line
+	18100 3350 19000 3350
+Wire Wire Line
+	19000 4400 19000 4200
+Wire Wire Line
+	18100 4400 19000 4400
+Wire Wire Line
+	1950 4100 1950 4900
+Wire Wire Line
+	1900 4800 2500 4800
+$Comp
+L Connector:Conn_01x02_Male J2
+U 1 1 5CDE4B86
+P 15850 5450
+F 0 "J2" H 15800 5650 50  0000 C CNN
+F 1 "PWR_BRIDGE2" H 15750 5550 50  0000 C CNN
+F 2 "YonaFootprints:TEDX_PWR_BRIDGE" H 15850 5450 50  0001 C CNN
+F 3 "~" H 15850 5450 50  0001 C CNN
+	1    15850 5450
+	1    0    0    -1
+$EndComp
+$Comp
+L power:+5V #PWR0127
+U 1 1 5CDE4B8C
+P 16050 5450
+F 0 "#PWR0127" H 16050 5300 50  0001 C CNN
+F 1 "+5V" H 16065 5623 50  0000 C CNN
+F 2 "" H 16050 5450 50  0001 C CNN
+F 3 "" H 16050 5450 50  0001 C CNN
+	1    16050 5450
+	1    0    0    -1
+$EndComp
+$Comp
+L power:GND #PWR0128
+U 1 1 5CDE4B92
+P 16050 5550
+F 0 "#PWR0128" H 16050 5300 50  0001 C CNN
+F 1 "GND" H 16055 5377 50  0000 C CNN
+F 2 "" H 16050 5550 50  0001 C CNN
+F 3 "" H 16050 5550 50  0001 C CNN
+	1    16050 5550
+	1    0    0    -1
+$EndComp
 $EndSCHEMATC
