File: FOutside/Strut.kicad_pcb (KiCad board)
At the start: 4 copper layers, 309.6 x 138.1 mm, 53 parts, among them J1 IN, J2 OUT

Commit message: First iteration of all struts
Parts:
- removed C17: 100NF, Capacitor_SMD:C_0805_2012Metric
- removed D17: WS2813, LED_SMD:LED_WS2812_PLCC6_5.0x5.0mm_P1.6mm
- removed R17: 330, Resistor_SMD:R_0805_2012Metric
- moved R16 56.7 mm to (313.7, 199.4), turned to 270 degrees
- moved R1 55.7 mm to (76.2, 199.4), turned to 270 degrees
- moved R9 55.7 mm to (209.6, 199.4), turned to 270 degrees
- moved J2 54.4 mm to (326.4, 196.8)
- moved C15 52.6 mm to (297.7, 199.4)
- moved C10 50.8 mm to (227.7, 199.4)
- moved C11 50.8 mm to (244.4, 199.4)
- moved C12 50.8 mm to (261.5, 199.4)
- moved C13 50.8 mm to (278.1, 199.4)
- moved C14 50.8 mm to (294.8, 199.4)
- moved C2 50.8 mm to (94.5, 199.4)
- moved C3 50.8 mm to (111.2, 199.4)
- moved C4 50.8 mm to (127.8, 199.4)
- moved C5 50.8 mm to (144.5, 199.4)
- moved C6 50.8 mm to (161.1, 199.4)
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Connections:
- J2 pad 2: Net-(D17-Pad3) -> Net-(D16-Pad3)
Routing:
- net Net-(D15-Pad3): track 36.1 -> 12.6 mm
- net GND: track 101.3 -> 119.7 mm, vias 20 -> 16
- net Net-(C17-Pad1): track 11.8 -> 0.00 mm
- net Net-(D17-Pad3): track 9.86 -> 0.00 mm, vias 1 -> 0
- net Net-(C1-Pad1): track 15.6 -> 6.56 mm
- net Net-(D16-Pad3): track 13.5 -> 4.95 mm
- net Net-(D1-Pad4): track 33.8 -> 25.5 mm
- net Net-(C15-Pad1): track 6.15 -> 11.2 mm, vias 0 -> 2
- net +5V: track 89.0 -> 93.7 mm, vias 19 -> 17
- net Net-(D10-Pad6): track 36.8 -> 32.6 mm
- net Net-(C9-Pad1): track 9.89 -> 7.09 mm, vias 2 -> 0
- net Net-(D1-Pad3): track 34.0 -> 31.9 mm
- net Net-(D14-Pad3): track 31.6 -> 33.5 mm
- net Net-(D10-Pad4): track 33.7 -> 32.6 mm
- net Net-(C16-Pad1): track 12.3 -> 11.6 mm, vias 0 -> 2
Other:
- outline, holes or cut-outs redrawn
