File: TestPanel1/TestPanel1.kicad_pcb (KiCad board)
At the start: 4 copper layers, 307.8 x 77.8 mm, 270 parts, among them J1 IN, J2 IN2, J3 OUT2, J4 PWR_BRIDGE, J5 OUT

Commit message: Second Prototype Run
Parts:
- removed the C1 at (87.8, 198.5)
- removed the C1 at (87.8, 182.0)
- removed the C10 at (237.8, 198.5)
- removed the C10 at (237.8, 182.0)
- removed the C11 at (254.5, 198.5)
- removed the C11 at (254.5, 182.0)
- removed the C12 at (271.1, 198.5)
- removed the C12 at (271.1, 182.0)
- removed the C13 at (287.8, 198.5)
- removed the C13 at (287.8, 182.0)
- removed the C14 at (304.5, 198.5)
- removed the C14 at (304.5, 182.0)
- removed the C15 at (321.1, 198.5)
- removed the C15 at (321.1, 182.0)
- removed the C2 at (104.5, 198.5)
- removed the C2 at (104.5, 182.0)
- removed the C3 at (121.1, 198.5)
- removed the C3 at (121.1, 182.0)
- removed the C4 at (137.8, 198.5)
- removed the C4 at (137.8, 182.0)
- removed the C5 at (154.5, 198.5)
- removed the C5 at (154.5, 182.0)
- removed the C6 at (171.1, 198.5)
- removed the C6 at (171.1, 182.0)
- removed the C7 at (187.8, 198.5)
- removed the C7 at (187.8, 182.0)
- removed the C8 at (204.5, 198.5)
- removed the C8 at (204.5, 182.0)
- removed the C9 at (221.1, 198.5)
- removed the C9 at (221.1, 182.0)
- removed the D1 at (85.7, 203.5)
- removed the D1 at (85.7, 187.0)
- removed the D10 at (235.7, 203.5)
- removed the D10 at (235.7, 187.0)
- removed the D11 at (252.4, 203.5)
- removed the D11 at (252.4, 187.0)
- removed the D12 at (269.0, 203.5)
- removed the D12 at (269.0, 187.0)
- removed the D13 at (285.7, 203.5)
- removed the D13 at (285.7, 187.0)
- removed the D14 at (302.4, 203.5)
- removed the D14 at (302.4, 187.0)
- removed the D15 at (319.0, 203.5)
- removed the D15 at (319.0, 187.0)
- removed the D2 at (102.4, 203.5)
- removed the D2 at (102.4, 187.0)
- removed the D3 at (119.0, 203.5)
- removed the D3 at (119.0, 187.0)
- removed the D4 at (135.7, 203.5)
- removed the D4 at (135.7, 187.0)
- removed the D5 at (152.4, 203.5)
- removed the D5 at (152.4, 187.0)
- removed the D6 at (169.0, 203.5)
- removed the D6 at (169.0, 187.0)
- removed the D7 at (185.7, 203.5)
- removed the D7 at (185.7, 187.0)
- removed the D8 at (202.4, 203.5)
- removed the D8 at (202.4, 187.0)
- removed the D9 at (219.0, 203.5)
- removed the D9 at (219.0, 187.0)
- removed the J1 at (79.5, 202.7)
- removed the J1 at (79.5, 186.2)
- removed the J2 at (331.5, 203.5)
- removed the J2 at (360.3, 140.0)
- removed the J2 at (331.5, 187.0)
- removed the J3 at (75.3, 203.5)
- removed the J3 at (72.8, 140.0)
- removed the J3 at (75.3, 187.0)
- removed the J3 at (72.8, 163.5)
- removed the J4 at (135.7, 197.5)
- removed the J4 at (252.4, 197.5)
- removed the J4 at (119.0, 197.5)
- removed the J4 at (119.0, 181.0)
- removed the J4 at (135.7, 181.0)
- removed the J4 at (152.4, 181.0)
- removed the J4 at (285.7, 181.0)
- removed the J4 at (269.0, 181.0)
- removed the J4 at (252.4, 181.0)
- removed the J4 at (235.7, 181.0)
- removed the J4 at (219.0, 181.0)
- removed the J4 at (269.0, 197.5)
- removed the J4 at (202.4, 181.0)
- removed the J4 at (185.7, 181.0)
- removed the J4 at (168.9, 181.0)
- removed the J4 at (219.0, 197.5)
- removed the J4 at (185.7, 197.5)
- removed the J4 at (202.4, 197.5)
- removed the J4 at (168.9, 197.5)
- removed the J4 at (285.7, 197.5)
- removed the J4 at (152.4, 197.5)
- removed the J4 at (235.7, 197.5)
- removed the J5 at (327.4, 202.7)
- removed the J5 at (356.1, 140.0)
- removed the J5 at (327.4, 186.2)
- removed JP1 (x4): DOUT2_ENABLE, Jumper:SolderJumper-2_P1.3mm_Open_TrianglePad1.0x1.5mm
- removed JP2 (x4): BOUT2_ENABLE, Jumper:SolderJumper-2_P1.3mm_Open_TrianglePad1.0x1.5mm
- removed the JP3 at (79.4, 197.0)
- removed the JP3 at (77.0, 134.0)
- removed the JP3 at (79.4, 180.5)
- removed the JP4 at (91.3, 197.7)
- removed the JP4 at (91.3, 181.2)
- removed the R1 at (83.6, 198.5)
- removed the R1 at (83.6, 182.0)
- removed the R10 at (233.6, 198.5)
- removed the R10 at (233.6, 182.0)
- removed the R11 at (250.3, 198.5)
- removed the R11 at (250.3, 182.0)
- removed the R12 at (267.0, 198.5)
- removed the R12 at (267.0, 182.0)
- removed the R13 at (283.6, 198.5)
- removed the R13 at (283.6, 182.0)
- removed the R14 at (300.3, 198.5)
- removed the R14 at (300.3, 182.0)
- removed the R15 at (317.0, 198.5)
- removed the R15 at (317.0, 182.0)
- removed the R2 at (100.3, 198.5)
- removed the R2 at (100.3, 182.0)
- removed the R3 at (117.0, 198.5)
- removed the R3 at (117.0, 182.0)
- removed the R4 at (133.6, 198.5)
- removed the R4 at (133.6, 182.0)
- removed the R5 at (150.3, 198.5)
- removed the R5 at (150.3, 182.0)
- removed the R6 at (167.0, 198.5)
- removed the R6 at (167.0, 182.0)
- removed the R7 at (183.6, 198.5)
- removed the R7 at (183.6, 182.0)
- removed the R8 at (200.3, 198.5)
- removed the R8 at (200.3, 182.0)
- removed the R9 at (217.0, 198.5)
- removed the R9 at (217.0, 182.0)
- added C1: .1uF, Capacitor_SMD:C_0603_1608Metric, F.Cu at (87.8, 198.5)
- added C1: .1uF, Capacitor_SMD:C_0603_1608Metric, F.Cu at (87.8, 182.0)
- added C10: .1uF, Capacitor_SMD:C_0603_1608Metric, F.Cu at (237.8, 198.5)
- added C10: .1uF, Capacitor_SMD:C_0603_1608Metric, F.Cu at (237.8, 182.0)
- added C11: .1uF, Capacitor_SMD:C_0603_1608Metric, F.Cu at (254.5, 198.5)
- added C11: .1uF, Capacitor_SMD:C_0603_1608Metric, F.Cu at (254.5, 182.0)
- added C12: .1uF, Capacitor_SMD:C_0603_1608Metric, F.Cu at (271.1, 198.5)
- added C12: .1uF, Capacitor_SMD:C_0603_1608Metric, F.Cu at (271.1, 182.0)
- added C13: .1uF, Capacitor_SMD:C_0603_1608Metric, F.Cu at (287.8, 198.5)
- added C13: .1uF, Capacitor_SMD:C_0603_1608Metric, F.Cu at (287.8, 182.0)
- added C14: .1uF, Capacitor_SMD:C_0603_1608Metric, F.Cu at (304.5, 198.5)
- added C14: .1uF, Capacitor_SMD:C_0603_1608Metric, F.Cu at (304.5, 182.0)
- added C15: .1uF, Capacitor_SMD:C_0603_1608Metric, F.Cu at (321.1, 198.5)
- added C15: .1uF, Capacitor_SMD:C_0603_1608Metric, F.Cu at (321.1, 182.0)
- added C2: .1uF, Capacitor_SMD:C_0603_1608Metric, F.Cu at (104.5, 198.5)
- added C2: .1uF, Capacitor_SMD:C_0603_1608Metric, F.Cu at (104.5, 182.0)
- added C3: .1uF, Capacitor_SMD:C_0603_1608Metric, F.Cu at (121.1, 198.5)
- added C3: .1uF, Capacitor_SMD:C_0603_1608Metric, F.Cu at (121.1, 182.0)
- added C4: .1uF, Capacitor_SMD:C_0603_1608Metric, F.Cu at (137.8, 198.5)
- added C4: .1uF, Capacitor_SMD:C_0603_1608Metric, F.Cu at (137.8, 182.0)
- added C5: .1uF, Capacitor_SMD:C_0603_1608Metric, F.Cu at (154.5, 198.5)
- added C5: .1uF, Capacitor_SMD:C_0603_1608Metric, F.Cu at (154.5, 182.0)
- added C6: .1uF, Capacitor_SMD:C_0603_1608Metric, F.Cu at (171.1, 198.5)
- added C6: .1uF, Capacitor_SMD:C_0603_1608Metric, F.Cu at (171.1, 182.0)
- added C7: .1uF, Capacitor_SMD:C_0603_1608Metric, F.Cu at (187.8, 198.5)
- added C7: .1uF, Capacitor_SMD:C_0603_1608Metric, F.Cu at (187.8, 182.0)
- added C8: .1uF, Capacitor_SMD:C_0603_1608Metric, F.Cu at (204.5, 198.5)
- added C8: .1uF, Capacitor_SMD:C_0603_1608Metric, F.Cu at (204.5, 182.0)
- added C9: .1uF, Capacitor_SMD:C_0603_1608Metric, F.Cu at (221.1, 198.5)
- added C9: .1uF, Capacitor_SMD:C_0603_1608Metric, F.Cu at (221.1, 182.0)
- added D1: WS2813, LED_SMD:LED_WS2812_PLCC6_5.0x5.0mm_P1.6mm, F.Cu at (85.7, 203.5)
- added D1: WS2813, LED_SMD:LED_WS2812_PLCC6_5.0x5.0mm_P1.6mm, F.Cu at (85.7, 187.0)
- added D10: WS2813, LED_SMD:LED_WS2812_PLCC6_5.0x5.0mm_P1.6mm, F.Cu at (235.7, 203.5)
- added D10: WS2813, LED_SMD:LED_WS2812_PLCC6_5.0x5.0mm_P1.6mm, F.Cu at (235.7, 187.0)
- added D11: WS2813, LED_SMD:LED_WS2812_PLCC6_5.0x5.0mm_P1.6mm, F.Cu at (252.4, 203.5)
- added D11: WS2813, LED_SMD:LED_WS2812_PLCC6_5.0x5.0mm_P1.6mm, F.Cu at (252.4, 187.0)
- added D12: WS2813, LED_SMD:LED_WS2812_PLCC6_5.0x5.0mm_P1.6mm, F.Cu at (269.0, 203.5)
- added D12: WS2813, LED_SMD:LED_WS2812_PLCC6_5.0x5.0mm_P1.6mm, F.Cu at (269.0, 187.0)
- added D13: WS2813, LED_SMD:LED_WS2812_PLCC6_5.0x5.0mm_P1.6mm, F.Cu at (285.7, 203.5)
- added D13: WS2813, LED_SMD:LED_WS2812_PLCC6_5.0x5.0mm_P1.6mm, F.Cu at (285.7, 187.0)
- added D14: WS2813, LED_SMD:LED_WS2812_PLCC6_5.0x5.0mm_P1.6mm, F.Cu at (302.4, 203.5)
- added D14: WS2813, LED_SMD:LED_WS2812_PLCC6_5.0x5.0mm_P1.6mm, F.Cu at (302.4, 187.0)
- added D15: WS2813, LED_SMD:LED_WS2812_PLCC6_5.0x5.0mm_P1.6mm, F.Cu at (319.0, 203.5)
- added D15: WS2813, LED_SMD:LED_WS2812_PLCC6_5.0x5.0mm_P1.6mm, F.Cu at (319.0, 187.0)
- added D2: WS2813, LED_SMD:LED_WS2812_PLCC6_5.0x5.0mm_P1.6mm, F.Cu at (102.4, 203.5)
- added D2: WS2813, LED_SMD:LED_WS2812_PLCC6_5.0x5.0mm_P1.6mm, F.Cu at (102.4, 187.0)
- added D3: WS2813, LED_SMD:LED_WS2812_PLCC6_5.0x5.0mm_P1.6mm, F.Cu at (119.0, 203.5)
- added D3: WS2813, LED_SMD:LED_WS2812_PLCC6_5.0x5.0mm_P1.6mm, F.Cu at (119.0, 187.0)
- added D4: WS2813, LED_SMD:LED_WS2812_PLCC6_5.0x5.0mm_P1.6mm, F.Cu at (135.7, 203.5)
- added D4: WS2813, LED_SMD:LED_WS2812_PLCC6_5.0x5.0mm_P1.6mm, F.Cu at (135.7, 187.0)
- added D5: WS2813, LED_SMD:LED_WS2812_PLCC6_5.0x5.0mm_P1.6mm, F.Cu at (152.4, 203.5)
- added D5: WS2813, LED_SMD:LED_WS2812_PLCC6_5.0x5.0mm_P1.6mm, F.Cu at (152.4, 187.0)
- added D6: WS2813, LED_SMD:LED_WS2812_PLCC6_5.0x5.0mm_P1.6mm, F.Cu at (169.0, 203.5)
- added D6: WS2813, LED_SMD:LED_WS2812_PLCC6_5.0x5.0mm_P1.6mm, F.Cu at (169.0, 187.0)
- added D7: WS2813, LED_SMD:LED_WS2812_PLCC6_5.0x5.0mm_P1.6mm, F.Cu at (185.7, 203.5)
- added D7: WS2813, LED_SMD:LED_WS2812_PLCC6_5.0x5.0mm_P1.6mm, F.Cu at (185.7, 187.0)
- added D8: WS2813, LED_SMD:LED_WS2812_PLCC6_5.0x5.0mm_P1.6mm, F.Cu at (202.4, 203.5)
- added D8: WS2813, LED_SMD:LED_WS2812_PLCC6_5.0x5.0mm_P1.6mm, F.Cu at (202.4, 187.0)
- added D9: WS2813, LED_SMD:LED_WS2812_PLCC6_5.0x5.0mm_P1.6mm, F.Cu at (219.0, 203.5)
- added D9: WS2813, LED_SMD:LED_WS2812_PLCC6_5.0x5.0mm_P1.6mm, F.Cu at (219.0, 187.0)
- added J1: IN, YonaFootprints:TEDX_INNER_4, F.Cu at (79.5, 202.7)
- added J1: IN, YonaFootprints:TEDX_INNER_4, F.Cu at (79.5, 186.2)
- added J2: IN2, YonaFootprints:TEDX_IN2, B.Cu at (331.5, 203.5)
- added J2: IN2, YonaFootprints:TEDX_IN2, B.Cu at (360.3, 163.5)
- added J2: IN2, YonaFootprints:TEDX_IN2, B.Cu at (331.5, 187.0)
- added J3: PWR_BRIDGE, YonaFootprints:TEDX_PWR_BRIDGE_TALL, B.Cu at (308.2, 170.5)
- added J3: PWR_BRIDGE, YonaFootprints:TEDX_PWR_BRIDGE_TALL, B.Cu at (191.5, 170.5)
- added J3: PWR_BRIDGE, YonaFootprints:TEDX_PWR_BRIDGE_TALL, B.Cu at (191.5, 160.5)
- added J3: PWR_BRIDGE, YonaFootprints:TEDX_PWR_BRIDGE_TALL, B.Cu at (308.2, 160.5)
- added J3: PWR_BRIDGE, YonaFootprints:TEDX_PWR_BRIDGE_TALL, B.Cu at (191.5, 137.0)
- added J3: PWR_BRIDGE, YonaFootprints:TEDX_PWR_BRIDGE_TALL, B.Cu at (191.5, 147.0)
- added J3: PWR_BRIDGE, YonaFootprints:TEDX_PWR_BRIDGE_TALL, B.Cu at (308.2, 147.0)
- added J3: PWR_BRIDGE, YonaFootprints:TEDX_PWR_BRIDGE_TALL, B.Cu at (308.2, 137.0)
- added J4: PWR_BRIDGE, YonaFootprints:TEDX_PWR_BRIDGE_TALL, B.Cu at (152.4, 200.3)
- added J4: PWR_BRIDGE, YonaFootprints:TEDX_PWR_BRIDGE_TALL, B.Cu at (269.0, 200.3)
- added J4: DAT_BRIDGE, YonaFootprints:TEDX_DAT_BRIDGE_TALL, B.Cu at (341.5, 160.5)
- added J4: DAT_BRIDGE, YonaFootprints:TEDX_DAT_BRIDGE_TALL, B.Cu at (341.5, 137.0)
- added J4: PWR_BRIDGE, YonaFootprints:TEDX_PWR_BRIDGE_TALL, B.Cu at (269.0, 183.8)
- added J4: PWR_BRIDGE, YonaFootprints:TEDX_PWR_BRIDGE_TALL, B.Cu at (152.4, 183.8)
- added J5: OUT, YonaFootprints:TEDX_INNER_4, F.Cu at (327.4, 202.7)
- added J5: OUT, YonaFootprints:TEDX_INNER_4, F.Cu at (356.1, 163.5)
- added J5: OUT, YonaFootprints:TEDX_INNER_4, F.Cu at (327.4, 186.2)
- added J6: DAT_BRIDGE, YonaFootprints:TEDX_DAT_BRIDGE_TALL, B.Cu at (302.4, 200.3)
- added J6: DAT_BRIDGE, YonaFootprints:TEDX_DAT_BRIDGE_TALL, B.Cu at (302.4, 183.8)
- added JP3: DOUT2_ENABLE, Jumper:SolderJumper-2_P1.3mm_Open_TrianglePad1.0x1.5mm, B.Cu at (79.4, 197.0)
- added JP3: DOUT2_ENABLE, Jumper:SolderJumper-2_P1.3mm_Open_TrianglePad1.0x1.5mm, B.Cu at (81.3, 169.3)
- added JP3: DOUT2_ENABLE, Jumper:SolderJumper-2_P1.3mm_Open_TrianglePad1.0x1.5mm, B.Cu at (81.3, 145.8)
- added JP4: BOUT2_ENABLE, Jumper:SolderJumper-2_P1.3mm_Open_TrianglePad1.0x1.5mm, B.Cu at (91.3, 197.7)
- added JP4: BOUT2_ENABLE, Jumper:SolderJumper-2_P1.3mm_Open_TrianglePad1.0x1.5mm, B.Cu at (91.3, 181.2)
- added R1: 330, Resistor_SMD:R_0603_1608Metric, F.Cu at (83.6, 198.5)
- added R1: 330, Resistor_SMD:R_0603_1608Metric, F.Cu at (83.6, 182.0)
- added R10: 330, Resistor_SMD:R_0603_1608Metric, F.Cu at (233.6, 198.5)
- added R10: 330, Resistor_SMD:R_0603_1608Metric, F.Cu at (233.6, 182.0)
- added R11: 330, Resistor_SMD:R_0603_1608Metric, F.Cu at (250.3, 198.5)
- added R11: 330, Resistor_SMD:R_0603_1608Metric, F.Cu at (250.3, 182.0)
- added R12: 330, Resistor_SMD:R_0603_1608Metric, F.Cu at (267.0, 198.5)
- added R12: 330, Resistor_SMD:R_0603_1608Metric, F.Cu at (267.0, 182.0)
- added R13: 330, Resistor_SMD:R_0603_1608Metric, F.Cu at (283.6, 198.5)
- added R13: 330, Resistor_SMD:R_0603_1608Metric, F.Cu at (283.6, 182.0)
- added R14: 330, Resistor_SMD:R_0603_1608Metric, F.Cu at (300.3, 198.5)
- added R14: 330, Resistor_SMD:R_0603_1608Metric, F.Cu at (300.3, 182.0)
- added R15: 330, Resistor_SMD:R_0603_1608Metric, F.Cu at (317.0, 198.5)
- added R15: 330, Resistor_SMD:R_0603_1608Metric, F.Cu at (317.0, 182.0)
- added R2: 330, Resistor_SMD:R_0603_1608Metric, F.Cu at (100.3, 198.5)
- added R2: 330, Resistor_SMD:R_0603_1608Metric, F.Cu at (100.3, 182.0)
- added R3: 330, Resistor_SMD:R_0603_1608Metric, F.Cu at (117.0, 198.5)
- added R3: 330, Resistor_SMD:R_0603_1608Metric, F.Cu at (117.0, 182.0)
- added R4: 330, Resistor_SMD:R_0603_1608Metric, F.Cu at (133.6, 198.5)
- added R4: 330, Resistor_SMD:R_0603_1608Metric, F.Cu at (133.6, 182.0)
- added R5: 330, Resistor_SMD:R_0603_1608Metric, F.Cu at (150.3, 198.5)
- added R5: 330, Resistor_SMD:R_0603_1608Metric, F.Cu at (150.3, 182.0)
- added R6: 330, Resistor_SMD:R_0603_1608Metric, F.Cu at (167.0, 198.5)
- added R6: 330, Resistor_SMD:R_0603_1608Metric, F.Cu at (167.0, 182.0)
- added R7: 330, Resistor_SMD:R_0603_1608Metric, F.Cu at (183.6, 198.5)
- added R7: 330, Resistor_SMD:R_0603_1608Metric, F.Cu at (183.6, 182.0)
- added R8: 330, Resistor_SMD:R_0603_1608Metric, F.Cu at (200.3, 198.5)
- added R8: 330, Resistor_SMD:R_0603_1608Metric, F.Cu at (200.3, 182.0)
- added R9: 330, Resistor_SMD:R_0603_1608Metric, F.Cu at (217.0, 198.5)
- added R9: 330, Resistor_SMD:R_0603_1608Metric, F.Cu at (217.0, 182.0)
- moved C16 23.5 mm to (335.3, 158.5)
- moved C16 23.5 mm to (335.3, 135.0)
- moved C17 23.5 mm to (352.0, 158.5)
- moved C17 23.5 mm to (352.0, 135.0)
- moved D16 23.5 mm to (333.2, 163.5)
- moved D16 23.5 mm to (333.2, 140.0)
- moved D17 23.5 mm to (349.9, 163.5)
- moved D17 23.5 mm to (349.9, 140.0)
- moved J2 23.5 mm to (360.3, 140.0)
- moved J5 23.5 mm to (356.1, 140.0)
- moved R16 23.5 mm to (331.1, 158.5)
- moved R16 23.5 mm to (331.1, 135.0)
- moved R17 23.5 mm to (347.8, 158.5)
- moved R17 23.5 mm to (347.8, 135.0)
- moved JP3 23.1 mm to (79.4, 180.5)
Routing:
- net Net-(J3-Pad1): track 1110.3 -> 0.00 mm, vias 10 -> 0
- net Net-(J3-Pad2): track 1095.0 -> 0.00 mm, vias 10 -> 0
- net GND: track 387.3 -> 254.8 mm
- net +5V: track 385.9 -> 288.5 mm, vias 136 -> 100
- net Net-(D15-Pad3): track 92.9 -> 73.4 mm, vias 8 -> 10
- net /DOUT: track 89.5 -> 98.8 mm, vias 6 -> 14
- net /DIN: track 131.4 -> 122.4 mm, vias 0 -> 4
- net /BOUT: track 140.4 -> 147.0 mm, vias 8 -> 6
- net Net-(D13-Pad3): track 134.2 -> 140.3 mm, vias 8 -> 12
- net Net-(D6-Pad3): track 132.5 -> 137.4 mm, vias 8 -> 12
- net Net-(D7-Pad3): track 132.3 -> 136.8 mm
- net Net-(D5-Pad3): track 132.6 -> 136.8 mm, vias 8 -> 12
- net Net-(D10-Pad4): track 132.1 -> 136.2 mm, vias 8 -> 12
- net Net-(D4-Pad3): track 132.2 -> 136.0 mm, vias 8 -> 12
- net Net-(D10-Pad6): track 132.2 -> 135.9 mm, vias 8 -> 12
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Other:
- board text added: "G"
- board text removed: "BK-OUT C/O ENABLE"
- board text removed: "DAT-OUT C/O ENABLE"
- board text removed: "OUT"
