File: TestPanel2/TestPanel2.kicad_pcb (KiCad board)
At the start: 4 copper layers, 250 x 40.5 mm, 402 parts, among them J1 IN, J2 MID, J3 MID, J4 MID, J5 OUT, J6 PWR_BRIDGE

Commit message: Second Prototype Run
Parts:
- removed the C1 at (91.4, 108.4)
- removed the C1 at (91.4, 74.4)
- removed the C1 at (91.4, 99.9)
- removed the C1 at (91.4, 91.4)
- removed the C1 at (91.4, 82.9)
- removed the C10 at (241.4, 108.4)
- removed the C10 at (241.4, 74.4)
- removed the C10 at (241.4, 99.9)
- removed the C10 at (241.4, 91.4)
- removed the C10 at (241.4, 82.9)
- removed the C12 at (263.3, 109.5)
- removed the C12 at (263.3, 75.5)
- removed the C12 at (263.3, 101.0)
- removed the C12 at (263.3, 92.5)
- removed the C12 at (263.3, 84.0)
- removed the C13 at (280.2, 109.6)
- removed the C13 at (280.2, 75.6)
- removed the C13 at (280.2, 101.1)
- removed the C13 at (280.2, 92.6)
- removed the C13 at (280.2, 84.1)
- removed the C14 at (296.9, 109.6)
- removed the C14 at (296.9, 75.6)
- removed the C14 at (296.9, 101.1)
- removed the C14 at (296.9, 92.6)
- removed the C14 at (296.9, 84.1)
- removed the C15 at (313.5, 109.6)
- removed the C15 at (313.5, 75.6)
- removed the C15 at (313.5, 101.1)
- removed the C15 at (313.5, 92.6)
- removed the C15 at (313.5, 84.1)
- removed the C3 at (124.7, 108.4)
- removed the C3 at (124.7, 74.4)
- removed the C3 at (124.7, 99.9)
- removed the C3 at (124.7, 91.4)
- removed the C3 at (124.7, 82.9)
- removed the J1 at (77.9, 108.6)
- removed the J1 at (77.9, 74.6)
- removed the J1 at (77.9, 100.1)
- removed the J1 at (77.9, 91.6)
- removed the J1 at (77.9, 83.1)
- removed the J5 at (324.9, 108.6)
- removed the J5 at (324.9, 74.6)
- removed the J5 at (324.9, 100.1)
- removed the J5 at (324.9, 91.6)
- removed the J5 at (324.9, 83.1)
- removed the J6 at (268.1, 105.4)
- removed the J6 at (151.4, 111.9)
- removed the J6 at (84.7, 79.9)
- removed the J6 at (101.4, 86.4)
- removed the J6 at (101.4, 79.9)
- removed the J6 at (151.4, 86.4)
- removed the J6 at (118.1, 86.4)
- removed the J6 at (134.7, 79.9)
- removed the J6 at (134.7, 86.1)
- removed the J6 at (118.1, 111.9)
- removed the J6 at (118.1, 79.9)
- removed the J6 at (151.4, 79.9)
- removed the J6 at (134.7, 105.4)
- removed the J6 at (268.1, 86.4)
- removed the J6 at (134.7, 111.6)
- removed the J6 at (118.1, 105.4)
- removed the J6 at (151.4, 105.4)
- removed the J6 at (84.7, 111.6)
- removed the J6 at (268.1, 111.9)
- removed the J6 at (268.1, 71.4)
- removed the J6 at (84.7, 77.6)
- removed the J6 at (84.7, 71.4)
- removed the J6 at (101.4, 77.9)
- removed the J6 at (101.4, 71.4)
- removed the J6 at (151.4, 77.9)
- removed the J6 at (118.1, 77.9)
- removed the J6 at (134.7, 71.4)
- removed the J6 at (134.7, 77.6)
- removed the J6 at (118.1, 71.4)
- removed the J6 at (151.4, 71.4)
- removed the J6 at (268.1, 77.9)
- removed the J6 at (268.1, 96.9)
- removed the J6 at (84.7, 103.1)
- removed the J6 at (84.7, 96.9)
- removed the J6 at (101.4, 103.4)
- removed the J6 at (101.4, 96.9)
- removed the J6 at (151.4, 103.4)
- removed the J6 at (118.1, 103.4)
- removed the J6 at (134.7, 96.9)
- removed the J6 at (134.7, 103.1)
- removed the J6 at (118.1, 96.9)
- removed the J6 at (151.4, 96.9)
- removed the J6 at (84.7, 105.4)
- removed the J6 at (268.1, 103.4)
- removed the J6 at (268.1, 88.4)
- removed the J6 at (84.7, 94.6)
- removed the J6 at (84.7, 88.4)
- removed the J6 at (101.4, 111.9)
- removed the J6 at (101.4, 94.9)
- removed the J6 at (101.4, 88.4)
- removed the J6 at (151.4, 94.9)
- removed the J6 at (118.1, 94.9)
- removed the J6 at (134.7, 88.4)
- removed the J6 at (134.7, 94.6)
- removed the J6 at (118.1, 88.4)
- removed the J6 at (151.4, 88.4)
- removed the J6 at (101.4, 105.4)
- removed the J6 at (268.1, 94.9)
- removed the J6 at (268.1, 79.9)
- removed the J6 at (84.7, 86.1)
- removed the R1 at (89.6, 108.4)
- removed the R1 at (89.6, 74.4)
- removed the R1 at (89.6, 99.9)
- removed the R1 at (89.6, 91.4)
- removed the R1 at (89.6, 82.9)
- removed the R10 at (239.6, 108.4)
- removed the R10 at (239.6, 74.4)
- removed the R10 at (239.6, 99.9)
- removed the R10 at (239.6, 91.4)
- removed the R10 at (239.6, 82.9)
- removed the R13 at (289.3, 109.6)
- removed the R13 at (289.3, 75.6)
- removed the R13 at (289.3, 101.1)
- removed the R13 at (289.3, 92.6)
- removed the R13 at (289.3, 84.1)
- removed the R14 at (305.9, 109.6)
- removed the R14 at (305.9, 75.6)
- removed the R14 at (305.9, 101.1)
- removed the R14 at (305.9, 92.6)
- removed the R14 at (305.9, 84.1)
- removed the R15 at (322.6, 109.6)
- removed the R15 at (322.6, 75.6)
- removed the R15 at (322.6, 101.1)
- removed the R15 at (322.6, 92.6)
- removed the R15 at (322.6, 84.1)
- removed the R3 at (123.0, 108.4)
- removed the R3 at (123.0, 74.4)
- removed the R3 at (123.0, 99.9)
- removed the R3 at (123.0, 91.4)
- removed the R3 at (123.0, 82.9)
- added C1: .1uF, Capacitor_SMD:C_0603_1608Metric, F.Cu at (91.5, 110.2)
- added C1: .1uF, Capacitor_SMD:C_0603_1608Metric, F.Cu at (91.5, 101.7)
- added C1: .1uF, Capacitor_SMD:C_0603_1608Metric, F.Cu at (91.5, 93.2)
- added C1: .1uF, Capacitor_SMD:C_0603_1608Metric, F.Cu at (91.5, 84.7)
- added C1: .1uF, Capacitor_SMD:C_0603_1608Metric, F.Cu at (91.5, 76.2)
- added C10: .1uF, Capacitor_SMD:C_0603_1608Metric, F.Cu at (244.9, 110.4)
- added C10: .1uF, Capacitor_SMD:C_0603_1608Metric, F.Cu at (244.9, 101.9)
- added C10: .1uF, Capacitor_SMD:C_0603_1608Metric, F.Cu at (244.9, 93.4)
- added C10: .1uF, Capacitor_SMD:C_0603_1608Metric, F.Cu at (244.9, 84.9)
- added C10: .1uF, Capacitor_SMD:C_0603_1608Metric, F.Cu at (244.9, 76.4)
- added C12: .1uF, Capacitor_SMD:C_0603_1608Metric, F.Cu at (262.7, 110.4)
- added C12: .1uF, Capacitor_SMD:C_0603_1608Metric, F.Cu at (262.7, 101.9)
- added C12: .1uF, Capacitor_SMD:C_0603_1608Metric, F.Cu at (262.7, 93.4)
- added C12: .1uF, Capacitor_SMD:C_0603_1608Metric, F.Cu at (262.7, 84.9)
- added C12: .1uF, Capacitor_SMD:C_0603_1608Metric, F.Cu at (262.7, 76.4)
- added C13: .1uF, Capacitor_SMD:C_0603_1608Metric, F.Cu at (280.2, 109.9)
- added C13: .1uF, Capacitor_SMD:C_0603_1608Metric, F.Cu at (280.2, 101.4)
- added C13: .1uF, Capacitor_SMD:C_0603_1608Metric, F.Cu at (280.2, 92.9)
- added C13: .1uF, Capacitor_SMD:C_0603_1608Metric, F.Cu at (280.2, 84.4)
- added C13: .1uF, Capacitor_SMD:C_0603_1608Metric, F.Cu at (280.2, 75.9)
- added C14: .1uF, Capacitor_SMD:C_0603_1608Metric, F.Cu at (296.9, 109.9)
- added C14: .1uF, Capacitor_SMD:C_0603_1608Metric, F.Cu at (296.9, 101.4)
- added C14: .1uF, Capacitor_SMD:C_0603_1608Metric, F.Cu at (296.9, 92.9)
- added C14: .1uF, Capacitor_SMD:C_0603_1608Metric, F.Cu at (296.9, 84.4)
- added C14: .1uF, Capacitor_SMD:C_0603_1608Metric, F.Cu at (296.9, 75.9)
- added C15: .1uF, Capacitor_SMD:C_0603_1608Metric, F.Cu at (313.5, 109.9)
- added C15: .1uF, Capacitor_SMD:C_0603_1608Metric, F.Cu at (313.5, 101.4)
- added C15: .1uF, Capacitor_SMD:C_0603_1608Metric, F.Cu at (313.5, 92.9)
- added C15: .1uF, Capacitor_SMD:C_0603_1608Metric, F.Cu at (313.5, 84.4)
- added C15: .1uF, Capacitor_SMD:C_0603_1608Metric, F.Cu at (313.5, 75.9)
- added C3: .1uF, Capacitor_SMD:C_0603_1608Metric, F.Cu at (129.0, 110.1)
- added C3: .1uF, Capacitor_SMD:C_0603_1608Metric, F.Cu at (129.0, 101.6)
- added C3: .1uF, Capacitor_SMD:C_0603_1608Metric, F.Cu at (129.0, 93.1)
- added C3: .1uF, Capacitor_SMD:C_0603_1608Metric, F.Cu at (129.0, 84.6)
- added C3: .1uF, Capacitor_SMD:C_0603_1608Metric, F.Cu at (129.0, 76.1)
- added J1: IN, YonaFootprints:6mmStripEnd, F.Cu at (77.6, 108.6)
- added J1: IN, YonaFootprints:6mmStripEnd, F.Cu at (77.6, 100.1)
- added J1: IN, YonaFootprints:6mmStripEnd, F.Cu at (77.6, 91.6)
- added J1: IN, YonaFootprints:6mmStripEnd, F.Cu at (77.6, 83.1)
- added J1: IN, YonaFootprints:6mmStripEnd, F.Cu at (77.6, 74.6)
- added J10: DAT_BRIDGE, YonaFootprints:TEDX_DAT_BRIDGE, B.Cu at (301.4, 107.9)
- added J10: DAT_BRIDGE, YonaFootprints:TEDX_DAT_BRIDGE, B.Cu at (301.4, 73.9)
- added J10: DAT_BRIDGE, YonaFootprints:TEDX_DAT_BRIDGE, B.Cu at (301.4, 111.9)
- added J10: DAT_BRIDGE, YonaFootprints:TEDX_DAT_BRIDGE, B.Cu at (301.4, 99.4)
- added J10: DAT_BRIDGE, YonaFootprints:TEDX_DAT_BRIDGE, B.Cu at (301.4, 103.4)
- added J10: DAT_BRIDGE, YonaFootprints:TEDX_DAT_BRIDGE, B.Cu at (301.4, 90.9)
- added J10: DAT_BRIDGE, YonaFootprints:TEDX_DAT_BRIDGE, B.Cu at (301.4, 94.9)
- added J10: DAT_BRIDGE, YonaFootprints:TEDX_DAT_BRIDGE, B.Cu at (301.4, 82.4)
- added J10: DAT_BRIDGE, YonaFootprints:TEDX_DAT_BRIDGE, B.Cu at (301.4, 86.4)
- added J10: DAT_BRIDGE, YonaFootprints:TEDX_DAT_BRIDGE, B.Cu at (301.4, 77.9)
- added J11: DAT_BRIDGE, YonaFootprints:TEDX_DAT_BRIDGE, B.Cu at (318.1, 107.9)
- added J11: DAT_BRIDGE, YonaFootprints:TEDX_DAT_BRIDGE, B.Cu at (318.1, 73.9)
- added J11: DAT_BRIDGE, YonaFootprints:TEDX_DAT_BRIDGE, B.Cu at (318.1, 111.9)
- added J11: DAT_BRIDGE, YonaFootprints:TEDX_DAT_BRIDGE, B.Cu at (318.1, 99.4)
- added J11: DAT_BRIDGE, YonaFootprints:TEDX_DAT_BRIDGE, B.Cu at (318.1, 103.4)
- added J11: DAT_BRIDGE, YonaFootprints:TEDX_DAT_BRIDGE, B.Cu at (318.1, 90.9)
- added J11: DAT_BRIDGE, YonaFootprints:TEDX_DAT_BRIDGE, B.Cu at (318.1, 94.9)
- added J11: DAT_BRIDGE, YonaFootprints:TEDX_DAT_BRIDGE, B.Cu at (318.1, 82.4)
- added J11: DAT_BRIDGE, YonaFootprints:TEDX_DAT_BRIDGE, B.Cu at (318.1, 86.4)
- added J11: DAT_BRIDGE, YonaFootprints:TEDX_DAT_BRIDGE, B.Cu at (318.1, 77.9)
- added J5: OUT, YonaFootprints:6mmStripEnd, F.Cu at (325.1, 108.6)
- added J5: OUT, YonaFootprints:6mmStripEnd, F.Cu at (325.1, 100.1)
- added J5: OUT, YonaFootprints:6mmStripEnd, F.Cu at (325.1, 91.6)
- added J5: OUT, YonaFootprints:6mmStripEnd, F.Cu at (325.1, 83.1)
- added J5: OUT, YonaFootprints:6mmStripEnd, F.Cu at (325.1, 74.6)
- added J6: PWR_BRIDGE, YonaFootprints:TEDX_PWR_BRIDGE, F.Cu at (243.1, 96.9)
- added J6: PWR_BRIDGE, YonaFootprints:TEDX_PWR_BRIDGE, F.Cu at (126.4, 96.9)
- added J6: PWR_BRIDGE, YonaFootprints:TEDX_PWR_BRIDGE, F.Cu at (126.4, 88.4)
- added J6: PWR_BRIDGE, YonaFootprints:TEDX_PWR_BRIDGE, F.Cu at (243.1, 88.4)
- added J6: PWR_BRIDGE, YonaFootprints:TEDX_PWR_BRIDGE, F.Cu at (243.1, 105.4)
- added J6: PWR_BRIDGE, YonaFootprints:TEDX_PWR_BRIDGE, F.Cu at (243.1, 79.9)
- added J6: PWR_BRIDGE, YonaFootprints:TEDX_PWR_BRIDGE, F.Cu at (126.4, 79.9)
- added J6: PWR_BRIDGE, YonaFootprints:TEDX_PWR_BRIDGE, F.Cu at (243.1, 71.4)
- added J6: PWR_BRIDGE, YonaFootprints:TEDX_PWR_BRIDGE, F.Cu at (126.4, 71.4)
- added J6: PWR_BRIDGE, YonaFootprints:TEDX_PWR_BRIDGE, F.Cu at (126.4, 105.4)
- added J7: DAT_BRIDGE, YonaFootprints:TEDX_DAT_BRIDGE, F.Cu at (93.1, 105.4)
- added J7: DAT_BRIDGE, YonaFootprints:TEDX_DAT_BRIDGE, B.Cu at (84.7, 86.4)
- added J7: DAT_BRIDGE, YonaFootprints:TEDX_DAT_BRIDGE, F.Cu at (93.1, 79.9)
- added J7: DAT_BRIDGE, YonaFootprints:TEDX_DAT_BRIDGE, B.Cu at (84.7, 79.9)
- added J7: DAT_BRIDGE, YonaFootprints:TEDX_DAT_BRIDGE, F.Cu at (93.1, 71.4)
- added J7: DAT_BRIDGE, YonaFootprints:TEDX_DAT_BRIDGE, B.Cu at (84.7, 77.9)
- added J7: DAT_BRIDGE, YonaFootprints:TEDX_DAT_BRIDGE, B.Cu at (84.7, 71.4)
- added J7: DAT_BRIDGE, YonaFootprints:TEDX_DAT_BRIDGE, B.Cu at (84.7, 111.9)
- added J7: DAT_BRIDGE, YonaFootprints:TEDX_DAT_BRIDGE, B.Cu at (84.7, 105.4)
- added J7: DAT_BRIDGE, YonaFootprints:TEDX_DAT_BRIDGE, B.Cu at (84.7, 96.9)
- added J7: DAT_BRIDGE, YonaFootprints:TEDX_DAT_BRIDGE, F.Cu at (93.1, 96.9)
- added J7: DAT_BRIDGE, YonaFootprints:TEDX_DAT_BRIDGE, B.Cu at (84.7, 103.4)
- added J7: DAT_BRIDGE, YonaFootprints:TEDX_DAT_BRIDGE, F.Cu at (93.1, 88.4)
- added J7: DAT_BRIDGE, YonaFootprints:TEDX_DAT_BRIDGE, B.Cu at (84.7, 94.9)
- added J7: DAT_BRIDGE, YonaFootprints:TEDX_DAT_BRIDGE, B.Cu at (84.7, 88.4)
- added J8: DAT_BRIDGE, YonaFootprints:TEDX_DAT_BRIDGE, B.Cu at (268.1, 107.8)
- added J8: DAT_BRIDGE, YonaFootprints:TEDX_DAT_BRIDGE, B.Cu at (268.1, 73.8)
- added J8: DAT_BRIDGE, YonaFootprints:TEDX_DAT_BRIDGE, B.Cu at (268.1, 111.9)
- added J8: DAT_BRIDGE, YonaFootprints:TEDX_DAT_BRIDGE, B.Cu at (268.1, 99.3)
- added J8: DAT_BRIDGE, YonaFootprints:TEDX_DAT_BRIDGE, B.Cu at (268.1, 103.4)
- added J8: DAT_BRIDGE, YonaFootprints:TEDX_DAT_BRIDGE, B.Cu at (268.1, 94.9)
- added J8: DAT_BRIDGE, YonaFootprints:TEDX_DAT_BRIDGE, B.Cu at (268.1, 90.8)
- added J8: DAT_BRIDGE, YonaFootprints:TEDX_DAT_BRIDGE, B.Cu at (268.1, 82.3)
- added J8: DAT_BRIDGE, YonaFootprints:TEDX_DAT_BRIDGE, B.Cu at (268.1, 86.4)
- added J8: DAT_BRIDGE, YonaFootprints:TEDX_DAT_BRIDGE, B.Cu at (268.1, 77.9)
- added J9: DAT_BRIDGE, YonaFootprints:TEDX_DAT_BRIDGE, B.Cu at (284.7, 111.9)
- added J9: DAT_BRIDGE, YonaFootprints:TEDX_DAT_BRIDGE, B.Cu at (284.7, 73.9)
- added J9: DAT_BRIDGE, YonaFootprints:TEDX_DAT_BRIDGE, B.Cu at (284.7, 107.9)
- added J9: DAT_BRIDGE, YonaFootprints:TEDX_DAT_BRIDGE, B.Cu at (284.7, 103.4)
- added J9: DAT_BRIDGE, YonaFootprints:TEDX_DAT_BRIDGE, B.Cu at (284.7, 99.4)
- added J9: DAT_BRIDGE, YonaFootprints:TEDX_DAT_BRIDGE, B.Cu at (284.7, 94.9)
- added J9: DAT_BRIDGE, YonaFootprints:TEDX_DAT_BRIDGE, B.Cu at (284.7, 90.9)
- added J9: DAT_BRIDGE, YonaFootprints:TEDX_DAT_BRIDGE, B.Cu at (284.7, 86.4)
- added J9: DAT_BRIDGE, YonaFootprints:TEDX_DAT_BRIDGE, B.Cu at (284.7, 82.4)
- added J9: DAT_BRIDGE, YonaFootprints:TEDX_DAT_BRIDGE, B.Cu at (284.7, 77.9)
- added R1: 330, Resistor_SMD:R_0603_1608Metric, F.Cu at (95.4, 110.2)
- added R1: 330, Resistor_SMD:R_0603_1608Metric, F.Cu at (95.4, 101.7)
- added R1: 330, Resistor_SMD:R_0603_1608Metric, F.Cu at (95.4, 93.2)
- added R1: 330, Resistor_SMD:R_0603_1608Metric, F.Cu at (95.4, 84.7)
- added R1: 330, Resistor_SMD:R_0603_1608Metric, F.Cu at (95.4, 76.2)
- added R10: 330, Resistor_SMD:R_0603_1608Metric, F.Cu at (241.4, 110.4)
- added R10: 330, Resistor_SMD:R_0603_1608Metric, F.Cu at (241.4, 101.9)
- added R10: 330, Resistor_SMD:R_0603_1608Metric, F.Cu at (241.4, 93.4)
- added R10: 330, Resistor_SMD:R_0603_1608Metric, F.Cu at (241.4, 84.9)
- added R10: 330, Resistor_SMD:R_0603_1608Metric, F.Cu at (241.4, 76.4)
- added R13: 330, Resistor_SMD:R_0603_1608Metric, F.Cu at (289.3, 109.9)
- added R13: 330, Resistor_SMD:R_0603_1608Metric, F.Cu at (289.3, 101.4)
- added R13: 330, Resistor_SMD:R_0603_1608Metric, F.Cu at (289.3, 92.9)
- added R13: 330, Resistor_SMD:R_0603_1608Metric, F.Cu at (289.3, 84.4)
- added R13: 330, Resistor_SMD:R_0603_1608Metric, F.Cu at (289.3, 75.9)
- added R14: 330, Resistor_SMD:R_0603_1608Metric, F.Cu at (305.9, 109.9)
- added R14: 330, Resistor_SMD:R_0603_1608Metric, F.Cu at (305.9, 101.4)
- added R14: 330, Resistor_SMD:R_0603_1608Metric, F.Cu at (305.9, 92.9)
- added R14: 330, Resistor_SMD:R_0603_1608Metric, F.Cu at (305.9, 84.4)
- added R14: 330, Resistor_SMD:R_0603_1608Metric, F.Cu at (305.9, 75.9)
- added R15: 330, Resistor_SMD:R_0603_1608Metric, F.Cu at (322.6, 109.9)
- added R15: 330, Resistor_SMD:R_0603_1608Metric, F.Cu at (322.6, 101.4)
- added R15: 330, Resistor_SMD:R_0603_1608Metric, F.Cu at (322.6, 92.9)
- added R15: 330, Resistor_SMD:R_0603_1608Metric, F.Cu at (322.6, 84.4)
- added R15: 330, Resistor_SMD:R_0603_1608Metric, F.Cu at (322.6, 75.9)
- added R3: 330, Resistor_SMD:R_0603_1608Metric, F.Cu at (125.7, 110.1)
- added R3: 330, Resistor_SMD:R_0603_1608Metric, F.Cu at (125.7, 101.6)
- added R3: 330, Resistor_SMD:R_0603_1608Metric, F.Cu at (125.7, 93.1)
- added R3: 330, Resistor_SMD:R_0603_1608Metric, F.Cu at (125.7, 84.6)
- added R3: 330, Resistor_SMD:R_0603_1608Metric, F.Cu at (125.7, 76.1)
Connections:
- C11 pad 1: (no net) -> Net-(C11-Pad1) (x5)
- C11 pad 2: (no net) -> GND (x5)
- C2 pad 1: (no net) -> Net-(C2-Pad1) (x5)
- C2 pad 2: (no net) -> GND (x5)
- C4 pad 1: (no net) -> Net-(C4-Pad1) (x5)
- C4 pad 2: (no net) -> GND (x5)
- C5 pad 1: (no net) -> Net-(C5-Pad1) (x5)
- C5 pad 2: (no net) -> GND (x5)
- C6 pad 1: (no net) -> Net-(C6-Pad1) (x5)
- C6 pad 2: (no net) -> GND (x5)
- C7 pad 1: (no net) -> Net-(C7-Pad1) (x5)
- C7 pad 2: (no net) -> GND (x5)
- C8 pad 1: (no net) -> Net-(C8-Pad1) (x5)
- C8 pad 2: (no net) -> GND (x5)
- C9 pad 1: (no net) -> Net-(C9-Pad1) (x5)
- C9 pad 2: (no net) -> GND (x5)
- D1 pad 1: (no net) -> Net-(C1-Pad1) (x5)
- D1 pad 2: (no net) -> +5V (x5)
- D1 pad 3: (no net) -> Net-(D1-Pad3) (x5)
- D1 pad 4: (no net) -> Net-(D1-Pad4) (x5)
- D1 pad 5: (no net) -> GND (x5)
- D1 pad 6: (no net) -> Net-(D1-Pad6) (x5)
- D10 pad 1: (no net) -> Net-(C10-Pad1) (x5)
- D10 pad 2: (no net) -> +5V (x5)
- D10 pad 3: (no net) -> Net-(D10-Pad3) (x5)
- D10 pad 4: (no net) -> Net-(D10-Pad4) (x5)
- D10 pad 5: (no net) -> GND (x5)
- D10 pad 6: (no net) -> Net-(D10-Pad6) (x5)
- D11 pad 1: (no net) -> Net-(C11-Pad1) (x5)
- D11 pad 2: (no net) -> +5V (x5)
- D11 pad 3: (no net) -> Net-(D11-Pad3) (x5)
- D11 pad 4: (no net) -> Net-(D10-Pad3) (x5)
- D11 pad 5: (no net) -> GND (x5)
- D11 pad 6: (no net) -> Net-(D10-Pad4) (x5)
- D12 pad 1: (no net) -> Net-(C12-Pad1) (x5)
- D12 pad 2: (no net) -> +5V (x5)
- D12 pad 3: (no net) -> Net-(D12-Pad3) (x5)
- D12 pad 4: (no net) -> Net-(D11-Pad3) (x5)
- D12 pad 5: (no net) -> GND (x5)
- D12 pad 6: (no net) -> Net-(D10-Pad3) (x5)
- D13 pad 1: (no net) -> Net-(C13-Pad1) (x5)
- D13 pad 2: (no net) -> +5V (x5)
- D13 pad 3: (no net) -> Net-(D13-Pad3) (x5)
- D13 pad 4: (no net) -> Net-(D12-Pad3) (x5)
- D13 pad 5: (no net) -> GND (x5)
- D13 pad 6: (no net) -> Net-(D11-Pad3) (x5)
- D14 pad 1: (no net) -> Net-(C14-Pad1) (x5)
- D14 pad 2: (no net) -> +5V (x5)
- D14 pad 3: (no net) -> Net-(D14-Pad3) (x5)
- D14 pad 4: (no net) -> Net-(D13-Pad3) (x5)
- D14 pad 5: (no net) -> GND (x5)
- D14 pad 6: (no net) -> Net-(D12-Pad3) (x5)
- D15 pad 1: (no net) -> Net-(C15-Pad1) (x5)
- D15 pad 2: (no net) -> +5V (x5)
- D15 pad 3: (no net) -> Net-(D15-Pad3) (x5)
- D15 pad 4: (no net) -> Net-(D14-Pad3) (x5)
- D15 pad 5: (no net) -> GND (x5)
- D15 pad 6: (no net) -> Net-(D13-Pad3) (x5)
- D2 pad 1: (no net) -> Net-(C2-Pad1) (x5)
- D2 pad 2: (no net) -> +5V (x5)
- D2 pad 3: (no net) -> Net-(D2-Pad3) (x5)
- D2 pad 4: (no net) -> Net-(D1-Pad3) (x5)
- D2 pad 5: (no net) -> GND (x5)
- D2 pad 6: (no net) -> Net-(D1-Pad4) (x5)
- D3 pad 1: (no net) -> Net-(C3-Pad1) (x5)
- D3 pad 2: (no net) -> +5V (x5)
- D3 pad 3: (no net) -> Net-(D3-Pad3) (x5)
- D3 pad 4: (no net) -> Net-(D2-Pad3) (x5)
- D3 pad 5: (no net) -> GND (x5)
- D3 pad 6: (no net) -> Net-(D1-Pad3) (x5)
- D4 pad 1: (no net) -> Net-(C4-Pad1) (x5)
- D4 pad 2: (no net) -> +5V (x5)
- D4 pad 3: (no net) -> Net-(D4-Pad3) (x5)
- D4 pad 4: (no net) -> Net-(D3-Pad3) (x5)
- D4 pad 5: (no net) -> GND (x5)
- D4 pad 6: (no net) -> Net-(D2-Pad3) (x5)
- D5 pad 1: (no net) -> Net-(C5-Pad1) (x5)
- D5 pad 2: (no net) -> +5V (x5)
- D5 pad 3: (no net) -> Net-(D5-Pad3) (x5)
- D5 pad 4: (no net) -> Net-(D4-Pad3) (x5)
- D5 pad 5: (no net) -> GND (x5)
- D5 pad 6: (no net) -> Net-(D3-Pad3) (x5)
- D6 pad 1: (no net) -> Net-(C6-Pad1) (x5)
- D6 pad 2: (no net) -> +5V (x5)
- D6 pad 3: (no net) -> Net-(D6-Pad3) (x5)
- D6 pad 4: (no net) -> Net-(D5-Pad3) (x5)
- D6 pad 5: (no net) -> GND (x5)
- D6 pad 6: (no net) -> Net-(D4-Pad3) (x5)
- D7 pad 1: (no net) -> Net-(C7-Pad1) (x5)
- D7 pad 2: (no net) -> +5V (x5)
- D7 pad 3: (no net) -> Net-(D7-Pad3) (x5)
- D7 pad 4: (no net) -> Net-(D6-Pad3) (x5)
- D7 pad 5: (no net) -> GND (x5)
- D7 pad 6: (no net) -> Net-(D5-Pad3) (x5)
- D8 pad 1: (no net) -> Net-(C8-Pad1) (x5)
- D8 pad 2: (no net) -> +5V (x5)
- D8 pad 3: (no net) -> Net-(D10-Pad6) (x5)
- D8 pad 4: (no net) -> Net-(D7-Pad3) (x5)
- D8 pad 5: (no net) -> GND (x5)
- D8 pad 6: (no net) -> Net-(D6-Pad3) (x5)
- D9 pad 1: (no net) -> Net-(C9-Pad1) (x5)
- D9 pad 2: (no net) -> +5V (x5)
- D9 pad 3: (no net) -> Net-(D10-Pad4) (x5)
- D9 pad 4: (no net) -> Net-(D10-Pad6) (x5)
- D9 pad 5: (no net) -> GND (x5)
- D9 pad 6: (no net) -> Net-(D7-Pad3) (x5)
- J2 pad 1: (no net) -> +5V (x5)
- J2 pad 2: (no net) -> Net-(D12-Pad3) (x5)
- J2 pad 3: (no net) -> Net-(D11-Pad3) (x5)
- J2 pad 4: (no net) -> GND (x5)
- J3 pad 1: (no net) -> +5V (x5)
- J3 pad 2: (no net) -> Net-(D13-Pad3) (x5)
- J3 pad 3: (no net) -> Net-(D12-Pad3) (x5)
- J3 pad 4: (no net) -> GND (x5)
- J4 pad 1: (no net) -> +5V (x5)
- J4 pad 2: (no net) -> Net-(D14-Pad3) (x5)
- J4 pad 3: (no net) -> Net-(D13-Pad3) (x5)
- J4 pad 4: (no net) -> GND (x5)
- J6 pad 1: (no net) -> +5V (x60)
- J6 pad 2: (no net) -> GND (x60)
- R11 pad 1: (no net) -> +5V (x5)
- R11 pad 2: (no net) -> Net-(C11-Pad1) (x5)
- R12 pad 1: (no net) -> +5V (x5)
- R12 pad 2: (no net) -> Net-(C12-Pad1) (x5)
- R2 pad 1: (no net) -> +5V (x5)
- R2 pad 2: (no net) -> Net-(C2-Pad1) (x5)
- R4 pad 1: (no net) -> +5V (x5)
- R4 pad 2: (no net) -> Net-(C4-Pad1) (x5)
- R5 pad 1: (no net) -> +5V (x5)
- R5 pad 2: (no net) -> Net-(C5-Pad1) (x5)
- R6 pad 1: (no net) -> +5V (x5)
- R6 pad 2: (no net) -> Net-(C6-Pad1) (x5)
- R7 pad 1: (no net) -> +5V (x5)
- R7 pad 2: (no net) -> Net-(C7-Pad1) (x5)
- R8 pad 1: (no net) -> +5V (x5)
- R8 pad 2: (no net) -> Net-(C8-Pad1) (x5)
- R9 pad 1: (no net) -> +5V (x5)
- R9 pad 2: (no net) -> Net-(C9-Pad1) (x5)
Routing:
- net (no net): track 4692.3 -> 0.00 mm, vias 350 -> 0
- net GND: track 0.00 -> 767.8 mm, vias 0 -> 120
- net +5V: track 0.00 -> 766.1 mm, vias 0 -> 60
- net Net-(D12-Pad3): track 0.00 -> 276.2 mm, vias 0 -> 20
- net Net-(D11-Pad3): track 0.00 -> 264.3 mm, vias 0 -> 15
- net Net-(D13-Pad3): track 0.00 -> 257.6 mm, vias 0 -> 20
- net Net-(D1-Pad6): track 0.00 -> 218.0 mm, vias 0 -> 15
- net Net-(D14-Pad3): track 0.00 -> 208.6 mm, vias 0 -> 20
- net Net-(D10-Pad3): track 0.00 -> 187.9 mm, vias 0 -> 20
- net Net-(D1-Pad3): track 0.00 -> 183.9 mm, vias 0 -> 10
- net Net-(D1-Pad4): track 0.00 -> 179.0 mm, vias 0 -> 20
- net Net-(D2-Pad3): track 0.00 -> 176.2 mm, vias 0 -> 10
- net Net-(D3-Pad3): track 0.00 -> 175.0 mm, vias 0 -> 15
- net Net-(D10-Pad4): track 0.00 -> 160.6 mm, vias 0 -> 10
- net Net-(D4-Pad3): track 0.00 -> 152.1 mm, vias 0 -> 10
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- added copper zone on In1.Cu, net +5V
- added copper zone on B.Cu, net GND
- added copper zone on In2.Cu, net GND
- removed copper zone on B.Cu, net (none)
- removed copper zone on In1.Cu, net (none)
- removed copper zone on In2.Cu, net (none)
Other:
- board text added: "5v"
- board text added: "BI"
- board text added: "BIN"
- board text added: "BO"
- board text added: "DI"
- board text added: "DIN"
- board text added: "DO"
- board text added: "G"
- board text added: "GND"
