File: EInside/EInside.sch (KiCad schematic (older format))
At the start: 59 parts, among them J1 IN, J2 IN2, J3 OUT2, J5 OUT

Commit message: Second Prototype Run
Parts:
- removed J3: OUT2, YonaFootprints:TEDX_IN2, symbol Connector:Conn_01x02_Female
- removed JP1: DOUT2_ENABLE, Jumper:SolderJumper-2_P1.3mm_Open_TrianglePad1.0x1.5mm, symbol Jumper:Jumper_2_Open
- removed JP2: BOUT2_ENABLE, Jumper:SolderJumper-2_P1.3mm_Open_TrianglePad1.0x1.5mm, symbol Jumper:Jumper_2_Open
- added J3: PWR_BRIDGE, YonaFootprints:TEDX_PWR_BRIDGE_TALL, symbol Connector:Conn_01x02_Male
- added J4: DAT_BRIDGE, YonaFootprints:TEDX_DAT_BRIDGE_TALL, symbol Connector:Conn_01x02_Female
Connections:
- net +5V: now also J3.1 (Pin_1)
- net BOUT: now also J4.2 (Pin_2)
- net DOUT: now also J4.1 (Pin_1)
- net GND: now also J3.2 (Pin_2)
Changed lines of the file:
@@
 EESchema Schematic File Version 4
 LIBS:EInside-cache
-LIBS:EOutside-cache
 EELAYER 29 0
 EELAYER END
@@
 	19200 4400 19850 4400
 Wire Wire Line
-	20400 4100 20450 4100
-Wire Wire Line
-	20650 4000 20500 4000
-Wire Wire Line
 	20650 4200 20550 4200
 Wire Wire Line
@@
 Text Label 20650 4100 2    50   ~ 0
 BOUT
-$Comp
-L Connector:Conn_01x02_Female J3
-U 1 1 5CF8C196
-P 21600 4550
-F 0 "J3" H 21628 4526 50  0000 L CNN
-F 1 "OUT2" H 21628 4435 50  0000 L CNN
-F 2 "YonaFootprints:TEDX_IN2" H 21600 4550 50  0001 C CNN
-F 3 "~" H 21600 4550 50  0001 C CNN
-	1    21600 4550
-	1    0    0    -1
-$EndComp
-Wire Wire Line
-	20450 4100 20450 4650
-Connection ~ 20450 4100
-Wire Wire Line
-	20450 4100 20650 4100
-Wire Wire Line
-	20500 4000 20500 4550
-Connection ~ 20500 4000
-Wire Wire Line
-	20500 4000 20150 4000
-$Comp
-L Jumper:Jumper_2_Open JP1
-U 1 1 5CFBB150
-P 21200 4550
-F 0 "JP1" H 21200 4785 50  0000 C CNN
-F 1 "DOUT2_ENABLE" H 21200 4694 50  0000 C CNN
-F 2 "Jumper:SolderJumper-2_P1.3mm_Open_TrianglePad1.0x1.5mm" H 21200 4550 50  0001 C CNN
-F 3 "~" H 21200 4550 50  0001 C CNN
-	1    21200 4550
-	1    0    0    -1
-$EndComp
-$Comp
-L Jumper:Jumper_2_Open JP2
-U 1 1 5CFBCECE
-P 21200 4650
-F 0 "JP2" H 21200 4500 50  0000 C CNN
-F 1 "BOUT2_ENABLE" H 21200 4400 50  0000 C CNN
-F 2 "Jumper:SolderJumper-2_P1.3mm_Open_TrianglePad1.0x1.5mm" H 21200 4650 50  0001 C CNN
-F 3 "~" H 21200 4650 50  0001 C CNN
-	1    21200 4650
-	1    0    0    -1
-$EndComp
-Wire Wire Line
-	20500 4550 21000 4550
-Wire Wire Line
-	20450 4650 21000 4650
 $Comp
 L Jumper:Jumper_2_Open JP3
@@
 Wire Wire Line
 	1150 4900 1300 4900
+Wire Wire Line
+	20150 4000 20600 4000
+Wire Wire Line
+	20400 4100 20500 4100
+$Comp
+L Connector:Conn_01x02_Male J3
+U 1 1 5CD29BC6
+P 12400 6050
+F 0 "J3" H 12508 6231 50  0000 C CNN
+F 1 "PWR_BRIDGE" H 12350 6150 50  0000 C CNN
+F 2 "YonaFootprints:TEDX_PWR_BRIDGE_TALL" H 12400 6050 50  0001 C CNN
+F 3 "~" H 12400 6050 50  0001 C CNN
+	1    12400 6050
+	1    0    0    -1
+$EndComp
+$Comp
+L power:+5V #PWR0125
+U 1 1 5CD29F28
+P 12650 6000
+F 0 "#PWR0125" H 12650 5850 50  0001 C CNN
+F 1 "+5V" H 12665 6173 50  0000 C CNN
+F 2 "" H 12650 6000 50  0001 C CNN
+F 3 "" H 12650 6000 50  0001 C CNN
+	1    12650 6000
+	1    0    0    -1
+$EndComp
+$Comp
+L power:GND #PWR0126
+U 1 1 5CD2A2A0
+P 12650 6200
+F 0 "#PWR0126" H 12650 5950 50  0001 C CNN
+F 1 "GND" H 12655 6027 50  0000 C CNN
+F 2 "" H 12650 6200 50  0001 C CNN
+F 3 "" H 12650 6200 50  0001 C CNN
+	1    12650 6200
+	1    0    0    -1
+$EndComp
+Wire Wire Line
+	12600 6050 12650 6050
+Wire Wire Line
+	12650 6050 12650 6000
+Wire Wire Line
+	12600 6150 12650 6150
+Wire Wire Line
+	12650 6150 12650 6200
+$Comp
+L Connector:Conn_01x02_Female J4
+U 1 1 5CD7C168
+P 20850 4950
+F 0 "J4" H 20878 4926 50  0000 L CNN
+F 1 "DAT_BRIDGE" H 20878 4835 50  0000 L CNN
+F 2 "YonaFootprints:TEDX_DAT_BRIDGE_TALL" H 20850 4950 50  0001 C CNN
+F 3 "~" H 20850 4950 50  0001 C CNN
+	1    20850 4950
+	1    0    0    -1
+$EndComp
+Wire Wire Line
+	20600 4000 20600 4950
+Wire Wire Line
+	20600 4950 20650 4950
+Connection ~ 20600 4000
+Wire Wire Line
+	20600 4000 20650 4000
+Wire Wire Line
+	20500 4100 20500 5050
+Wire Wire Line
+	20500 5050 20650 5050
+Connection ~ 20500 4100
+Wire Wire Line
+	20500 4100 20650 4100
 $EndSCHEMATC

Commit message: Before changing Outside Struts to not have connectors
Parts:
- removed J2: IN2, YonaFootprints:TEDX_IN2, symbol Connector:Conn_01x02_Male
- removed JP3: DOUT2_ENABLE, Jumper:SolderJumper-2_P1.3mm_Open_TrianglePad1.0x1.5mm, symbol Jumper:Jumper_2_Open
- removed JP4: BOUT2_ENABLE, Jumper:SolderJumper-2_P1.3mm_Open_TrianglePad1.0x1.5mm, symbol Jumper:Jumper_2_Open
Changed lines of the file:
@@
 	20650 3350 20650 3900
 Connection ~ 20300 3350
-$Comp
-L Connector:Conn_01x02_Male J2
-U 1 1 5CEC36A1
-P 950 4800
-F 0 "J2" H 1058 4981 50  0000 C CNN
-F 1 "IN2" H 1058 4890 50  0000 C CNN
-F 2 "YonaFootprints:TEDX_IN2" H 950 4800 50  0001 C CNN
-F 3 "~" H 950 4800 50  0001 C CNN
-	1    950  4800
-	1    0    0    -1
-$EndComp
-Wire Wire Line
-	1700 4800 1900 4800
-Wire Wire Line
-	1900 4800 1900 4350
-Connection ~ 1900 4350
-Wire Wire Line
-	1950 4100 1950 4900
-Wire Wire Line
-	1950 4900 1700 4900
-Connection ~ 1950 4100
 Wire Wire Line
 	1850 3900 1550 3900
@@
 Text Label 20650 4100 2    50   ~ 0
 BOUT
-$Comp
-L Jumper:Jumper_2_Open JP3
-U 1 1 5CFF526D
-P 1500 4800
-F 0 "JP3" H 1500 5035 50  0000 C CNN
-F 1 "DOUT2_ENABLE" H 1500 4944 50  0000 C CNN
-F 2 "Jumper:SolderJumper-2_P1.3mm_Open_TrianglePad1.0x1.5mm" H 1500 4800 50  0001 C CNN
-F 3 "~" H 1500 4800 50  0001 C CNN
-	1    1500 4800
-	-1   0    0    -1
-$EndComp
-$Comp
-L Jumper:Jumper_2_Open JP4
-U 1 1 5CFF5273
-P 1500 4900
-F 0 "JP4" H 1500 4750 50  0000 C CNN
-F 1 "BOUT2_ENABLE" H 1500 4650 50  0000 C CNN
-F 2 "Jumper:SolderJumper-2_P1.3mm_Open_TrianglePad1.0x1.5mm" H 1500 4900 50  0001 C CNN
-F 3 "~" H 1500 4900 50  0001 C CNN
-	1    1500 4900
-	-1   0    0    -1
-$EndComp
 Connection ~ 3800 3350
 Connection ~ 3800 4400
@@
 Connection ~ 19200 4400
 Wire Wire Line
-	1300 4800 1150 4800
-Wire Wire Line
-	1150 4900 1300 4900
-Wire Wire Line
 	20150 4000 20600 4000
