File: EInside/EInside.kicad_pcb (KiCad board)
At the start: 2 copper layers, 307.7 x 21.4 mm, 59 parts, among them J1 IN, J2 IN2, J3 OUT2, J5 OUT

Commit message: Second Prototype Run
Parts:
- removed the J3 at (59.2, 148.2)
- removed JP1: DOUT2_ENABLE, Jumper:SolderJumper-2_P1.3mm_Open_TrianglePad1.0x1.5mm
- removed JP2: BOUT2_ENABLE, Jumper:SolderJumper-2_P1.3mm_Open_TrianglePad1.0x1.5mm
- added J3: PWR_BRIDGE, YonaFootprints:TEDX_PWR_BRIDGE_TALL, B.Cu at (177.9, 145.2)
- added J3: PWR_BRIDGE, YonaFootprints:TEDX_PWR_BRIDGE_TALL, B.Cu at (177.9, 155.2)
- added J3: PWR_BRIDGE, YonaFootprints:TEDX_PWR_BRIDGE_TALL, B.Cu at (294.6, 155.2)
- added J3: PWR_BRIDGE, YonaFootprints:TEDX_PWR_BRIDGE_TALL, B.Cu at (294.6, 145.2)
- added J4: DAT_BRIDGE, YonaFootprints:TEDX_DAT_BRIDGE_TALL, B.Cu at (327.9, 145.2)
- moved JP3 12.6 mm to (67.7, 154.1), turned to 180 degrees
Routing:
- net Net-(J3-Pad1): track 290.5 -> 0.00 mm, vias 1 -> 0
- net Net-(J3-Pad2): track 287.4 -> 0.00 mm, vias 1 -> 0
- net +5V: track 52.4 -> 76.9 mm, vias 33 -> 34
- net Net-(D15-Pad3): track 46.4 -> 36.7 mm, vias 4 -> 5
- net /DOUT: track 28.7 -> 20.6 mm, vias 2 -> 3
- net /DIN: track 33.1 -> 30.9 mm, vias 0 -> 2
- net Net-(D13-Pad3): track 34.2 -> 36.1 mm, vias 2 -> 4
- net /BOUT: track 32.6 -> 31.5 mm, vias 3 -> 2
- net Net-(D6-Pad3): track 34.2 -> 35.3 mm, vias 2 -> 4
- net Net-(D7-Pad3): track 34.2 -> 35.1 mm
- net Net-(D10-Pad4): track 34.2 -> 35.0 mm, vias 2 -> 4
- net Net-(D4-Pad3): track 34.2 -> 34.9 mm, vias 2 -> 4
- net /BIN: track 11.6 -> 12.2 mm
- net Net-(D11-Pad3): track 34.2 -> 34.8 mm, vias 2 -> 4
- net Net-(D1-Pad3): track 34.2 -> 34.8 mm, vias 2 -> 4
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Other:
- outline, holes or cut-outs redrawn
- board text added: "BIN"
- board text added: "BOUT"
- board text added: "DIN"
- board text added: "DOUT"
- board text added: "G"
- board text removed: "BK-OUT C/O ENABLE"
- board text removed: "DAT-OUT C/O ENABLE"
- board text removed: "OUT"

Commit message: Before changing Outside Struts to not have connectors
Parts:
- removed J2: IN2, YonaFootprints:TEDX_IN2
- removed JP3: DOUT2_ENABLE, Jumper:SolderJumper-2_P1.3mm_Open_TrianglePad1.0x1.5mm
- removed JP4: BOUT2_ENABLE, Jumper:SolderJumper-2_P1.3mm_Open_TrianglePad1.0x1.5mm
- added J4: DAT_BRIDGE, YonaFootprints:TEDX_DAT_BRIDGE_TALL, B.Cu at (77.9, 155.2)
- moved J3 66.7 mm to (227.9, 155.2)
- moved J3 66.7 mm to (111.3, 155.2)
Routing:
- net Net-(J2-Pad2): track 288.3 -> 0.00 mm, vias 1 -> 0
- net Net-(J2-Pad1): track 286.0 -> 0.00 mm, vias 1 -> 0
- net +5V: track 76.9 -> 61.7 mm
- net /BIN: track 12.2 -> 4.15 mm, vias 1 -> 0
- net /DIN: track 30.9 -> 25.3 mm
- net Net-(D13-Pad3): track 36.1 -> 34.1 mm
- net /BOUT: track 31.5 -> 32.7 mm
- net Net-(D10-Pad4): track 35.0 -> 36.2 mm
- net Net-(D6-Pad3): track 35.3 -> 36.3 mm
Other:
- outline, holes or cut-outs redrawn
- board text added: "B"
- board text added: "DO"
- board text added: "NO-CONN"
- board text removed: "BK"
- board text removed: "BK-IN C/O ENABLE"
- board text removed: "DAT"
- board text removed: "DAT-IN C/O ENABLE"
- board text removed: "IN"

Commit message: Prototype v4
Routing:
- net Net-(D2-Pad3): track 34.3 -> 37.2 mm
- net Net-(D10-Pad4): track 36.2 -> 38.5 mm
- net Net-(D15-Pad3): track 36.7 -> 37.4 mm
Other:
- outline, holes or cut-outs redrawn
