File: AInside/AInside.kicad_pcb (KiCad board)
At the start: 4 copper layers, 231.2 x 14.2 mm, 38 parts, among them J1 A_IN, J2 A_OUT

Commit message: Prototype v4
Parts:
- removed the J2 at (256.5, 34.2)
- added J2: PWR_BRIDGE2, YonaFootprints:TEDX_PWR_BRIDGE, B.Cu at (227.8, 152.0)
- added J2: PWR_BRIDGE2, YonaFootprints:TEDX_PWR_BRIDGE, B.Cu at (111.2, 152.0)
- added J4: PWR_BRIDGE, YonaFootprints:TEDX_PWR_BRIDGE_TALL, B.Cu at (211.3, 145.0)
- added J4: PWR_BRIDGE, YonaFootprints:TEDX_PWR_BRIDGE_TALL, B.Cu at (94.6, 145.0)
- added J5: OUT, YonaFootprints:TEDX_INNER_4, F.Cu at (261.3, 147.5)
- added J6: DAT_BRIDGE, YonaFootprints:TEDX_DAT_BRIDGE_TALL, B.Cu at (244.6, 145.0)
- added JP3: CO_DIN_ENABLE, Jumper:SolderJumper-2_P1.3mm_Open_TrianglePad1.0x1.5mm, F.Cu at (54.5, 146.2)
- added JP4: CO_BIN_ENABLE, Jumper:SolderJumper-2_P1.3mm_Open_TrianglePad1.0x1.5mm, F.Cu at (54.5, 149.0)
- added REF**: TEDX_DAT_BRIDGE, YonaFootprints:TEDX_DAT_BRIDGE, B.Cu at (77.9, 152.0)
- C1, C10, C11, C12, C2, C3, C4, C5, C6, C7, C8, C9: value 100NF -> .1uF; footprint Capacitor_SMD:C_0805_2012Metric -> Capacitor_SMD:C_0603_1608Metric
- J1: value A_IN -> IN; footprint YonaFootprints:1x3_18awgWireSolderPad-InsideStrut-IN-Edge -> YonaFootprints:TEDX_INNER_4
- R1, R10, R11, R12, R2, R3, R4, R5, R6, R7, R8, R9: footprint Resistor_SMD:R_0805_2012Metric -> Resistor_SMD:R_0603_1608Metric
- moved J1 113.5 mm to (63.4, 147.5)
- moved D12 113.2 mm to (252.9, 148.2)
- moved D11 113.2 mm to (236.3, 148.2)
- moved D10 113.2 mm to (219.6, 148.2)
- moved D9 113.2 mm to (202.9, 148.2)
- moved D8 113.2 mm to (186.3, 148.2)
- moved D7 113.2 mm to (169.6, 148.2)
- moved D6 113.2 mm to (152.9, 148.2)
- moved D5 113.2 mm to (136.3, 148.2)
- moved D4 113.2 mm to (119.6, 148.2)
- moved D3 113.2 mm to (102.9, 148.2)
- moved D2 113.2 mm to (86.3, 148.2)
- moved D1 113.2 mm to (69.6, 148.2)
- moved C6 112.4 mm to (155.0, 143.2)
- moved C12 112.4 mm to (255.0, 143.2), turned to 0 degrees
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Connections:
- net Net-(D1-Pad4) renamed /DIN
- net Net-(D11-Pad3) renamed /BOUT
- D1 pad 6: GND -> /BIN
- D12 pad 3: Net-(D12-Pad3) -> /DOUT
- J1 pad 3: GND -> /BIN
Routing:
- net /CO_BIN: track 0.00 -> 228.7 mm, vias 0 -> 3
- net /CO_DIN: track 0.00 -> 218.5 mm, vias 0 -> 3
- net +5V: track 64.8 -> 99.1 mm, vias 11 -> 13
- net GND: track 81.0 -> 64.6 mm, vias 12 -> 27
- net /DOUT: track 0.00 -> 15.4 mm, vias 0 -> 3
- net /BIN: track 0.00 -> 12.7 mm
- net /BOUT: track 11.8 -> 22.1 mm, vias 0 -> 2
- net Net-(C1-Pad1): track 5.60 -> 12.4 mm
- net Net-(D12-Pad3): track 5.78 -> 0.00 mm
- net /DIN: track 25.1 -> 30.6 mm, vias 0 -> 2
- net Net-(C2-Pad1): track 5.93 -> 11.4 mm
- net Net-(C10-Pad1): track 5.93 -> 11.4 mm
- net Net-(C8-Pad1): track 5.93 -> 10.5 mm
- net Net-(C3-Pad1): track 5.93 -> 10.5 mm
- net Net-(C4-Pad1): track 5.93 -> 10.5 mm
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- removed copper zone on In2.Cu, net +5V
- removed copper zone on In1.Cu, net GND
Other:
- board size 231.2 x 14.2 mm -> 231.2 x 14.3 mm
- copper layers 4 -> 2
- board text added: "5v"
- board text added: "BIN"
- board text added: "BOUT"
- board text added: "C/O BIN"
- board text added: "C/O DIN"
- board text added: "CO"
- board text added: "DIN"
- board text added: "DOUT"
- board text added: "GND"
