File: AInside/AInside.sch (KiCad schematic (older format))
At the start: 38 parts, among them J1 A_IN, J2 A_OUT

Commit message: Prototype v4
Parts:
- removed J1: A_IN, YonaFootprints:1x3_18awgWireSolderPad-InsideStrut-IN-Edge, symbol Connector:Conn_01x03_Male
- removed J2: A_OUT, YonaFootprints:1x3_18awgWireSolderPad-InsideStrut-OUT-Edge, symbol Connector:Conn_01x03_Female
- added J1: IN, YonaFootprints:TEDX_INNER_4, symbol Connector:Conn_01x04_Male
- added J2: PWR_BRIDGE2, YonaFootprints:TEDX_PWR_BRIDGE, symbol Connector:Conn_01x02_Male
- added J4: PWR_BRIDGE, YonaFootprints:TEDX_PWR_BRIDGE_TALL, symbol Connector:Conn_01x02_Male
- added J5: OUT, YonaFootprints:TEDX_INNER_4, symbol Connector:Conn_01x04_Female
- added J6: DAT_BRIDGE, YonaFootprints:TEDX_DAT_BRIDGE_TALL, symbol Connector:Conn_01x02_Male
- added JP3: CO_DIN_ENABLE, Jumper:SolderJumper-2_P1.3mm_Open_TrianglePad1.0x1.5mm, symbol Jumper:Jumper_2_Open
- added JP4: CO_BIN_ENABLE, Jumper:SolderJumper-2_P1.3mm_Open_TrianglePad1.0x1.5mm, symbol Jumper:Jumper_2_Open
- C1, C10, C11, C12, C2, C3, C4, C5, C6, C7, C8, C9: value 100NF -> .1uF; footprint Capacitor_SMD:C_0805_2012Metric -> Capacitor_SMD:C_0603_1608Metric
- R1, R10, R11, R12, R2, R3, R4, R5, R6, R7, R8, R9: footprint Resistor_SMD:R_0805_2012Metric -> Resistor_SMD:R_0603_1608Metric
Connections:
- net labels added: BIN, BOUT, CO_BIN, CO_DIN, DIN, DOUT
- wire segments 207 -> 210
Other:
- note added: "A Strut\n12 LEDs\nx4"
- note removed: "A Strut\n12 LEDs\nx3"
